File: pcb/cyclops_r3/cyclops_r3.brd (EAGLE design)
At the start: 132.2 x 81.4 mm, 57 parts, among them IC2 317, IC3 REF02Z, IC5 LM324N, Q1 2N5087

Commit message: Updates to cyclops_r3 PCB.
Parts:
- removed EXT_CTL_K: SCREW3, HOSS:SCREW3
- removed I/O_BLOCK: SCREW5, HOSS:SCREW5
- removed LED+, LED-: BANANA_TO_BOARD, HOSS:BANANA_TO_BOARD
- removed LED_OUT: SCREW4, HOSS:SCREW4
- removed N-MOSFET: (no value), transistor-power:TO220BH
- removed V_CTL, V_CURR, V_PD, V_REF: 1-227161-0, con-coax:AMP_227161
- added IC1: 317TO263, cyclops:TO-263
- added U$2: ARDUINO_R3_ICSP, adafruit:ARDUINOR3_ICSP
- added U$3: SCREW2, cyclops:SCREW2
- IC5: value LM324N -> LM324D; device linear:DIL14 -> linear:SO14
Connections:
- new net 3V: U$2.3V
- new net 5V: U$2.+5V
- new net GND$1: U$2.GND$1
- new net GND$2: U$2.GND$2
- new net N$16: JP2.2
- new net N$66: U$2.MOSI
- new net N$67: U$2.RESET$1
- new net N$68: U$2.GND$3
- new net N$70: IC1.3, U$3.P$1
- new net VIN: U$2.VIN
- net GND: now also U$2.GND; no longer I/O_BLOCK.P$1, LED_OUT.P$1, V_CTL.2, V_CURR.2, V_PD.2, V_REF.2
- net N$10: no longer I/O_BLOCK.P$2, V_CTL.1
- net N$18: no longer I/O_BLOCK.P$3, V_REF.1
- net N$2: no longer N-MOSFET.S
- net N$21: now also U$2.5V; no longer LED-.P$1, LED_OUT.P$3, N-MOSFET.D
- net N$25: now also U$2.MISO; no longer EXT_CTL_K.P$1, JP2.2
- net N$26: now also U$2.SCK; no longer EXT_CTL_K.P$3, JP2.1
- net N$29: no longer N-MOSFET.G
- net N$4: no longer I/O_BLOCK.P$4, V_CURR.1
- net N$5: no longer I/O_BLOCK.P$5, V_PD.1
- net N$8: no longer EXT_CTL_K.P$2
- net P_12V: no longer LED_OUT.P$2
- net P_SUP: no longer LED+.P$1, LED_OUT.P$4
Routing:
- net N$21: track 90.9 -> 0.00 mm
- net P_SUP: track 53.6 -> 0.00 mm
- net GND: track 83.7 -> 78.2 mm

Commit message: Started designing the circuit.
Parts:
- removed GND1, V_IN1: BANANA_TO_BOARD, HOSS:BANANA_TO_BOARD
- removed MECH1, MECH2, MECH3, POW1: (no value), jumper:JP2Q
- removed POW2: SCREW2, HOSS:SCREW2
- removed Q1: 2N5087, transistor-pnp:TO92
- removed Q2: (no value), transistor-power:TO220BH
- removed R1, R5, R6: 1.5k, HOSS:0207/7
- removed U$1: FUSE >2A, HOSS:NXT-FUSE
- removed U$3: SCREW2, cyclops:SCREW2
- added C1: 10uF, cyclops:0805
- added C10, C13: 1uF, cyclops:1206-POL
- added C11: 10uF, cyclops:1206-POL
- added C12: 47uF, cyclops:153CLV-0807
- added C8: 0.1uF, cyclops:0805
- added D1, D2: S1B-13-F, cyclops:SMA-DO214AC
- added DAC: MCP4921SOIC, cyclops:SO08
- added POWER: SCREW2, cyclops:SCREW2
- added R11: 240k, cyclops:0603
- added R7: 1.8k, cyclops:0603
- added S1: 219-04, cyclops:CTS-219-04
- C9: value 10u -> 1uF; device rcl:C025-024X044 -> cyclops:0603
- IC1: value 317TO263 -> 317-N
- U$2: device adafruit:ARDUINOR3_ICSP -> cyclops:ARDUINOR3_ICSP
- moved C9 108.1 mm to (-39.4, -134.6)
- moved IC1 25.2 mm to (-17.8, -108.3), turned to 90 degrees
Connections:
- removed net N$21: U$2.5V
- removed net N$25: U$2.MISO
- removed net N$26: U$2.SCK
- removed net N$30: Q1.1, Q2.G, R1.1, R5.2
- removed net N$31: Q1.2, Q2.S, R6.1
- removed net N$61: POW1.1, U$1.P$1, U$1.P$2
- removed net N$66: U$2.MOSI
- removed net N$67: U$2.RESET$1
- removed net N$68: U$2.GND$3
- removed net N$70: IC1.3, U$3.P$1
- removed net P_SUP_BEFORE: Q1.3, R1.2, R6.2, U$1.P$4, U$1.P$53
- new net +12V: C12.+, C13.+, D1.A, D2.C, IC1.2, IC1.4, R11.2
- new net +15V: C10.+, D1.C, IC1.3, POWER.P$1
- new net +5V: C8.1, C9.1, DAC.1, U$2.5V
- new net CS: DAC.2, S1.1, S1.2, S1.3, S1.4
- new net CS0: S1.8, U$2.D1
- new net CS1: S1.7, U$2.D2
- new net CS2: S1.6, U$2.D3
- new net CS3: S1.5, U$2.D4
- new net DACA: DAC.8
- new net LDAC: DAC.5, U$2.D0
- new net N$72: C11.+, D2.A, IC1.1, R11.1, R7.2
- new net REFA: C1.1, DAC.6
- new net SCLK: DAC.3, U$2.SCK
- new net SDI: DAC.4, U$2.MOSI
- net GND: now also C1.2, C10.-, C11.-, C12.-, C13.-, C8.2, C9.2, DAC.7, POWER.P$2, R7.1, U$2.GND$3; no longer C9.1, GND1.P$1, POW1.4, POW2.P$1, R5.1
- net P_SUP: no longer C9.2, Q2.D
Routing:
- net GND: track 78.2 -> 76.4 mm

Commit message: More work on the circuit schematic.
Parts:
- removed +12V, GND2: BANANA_TO_BOARD, HOSS:BANANA_TO_BOARD
- removed C6: 0.1uF, rcl:C050-024X044
- removed IC2: 317, HOSS:TO220BH
- removed IC3: REF02Z, linear:DIL08
- removed IMEAS_K: 10k, HOSS:RJ6S
- removed JP1: (no value), jumper:JP3Q
- removed ON: (no value), led:LED3MM
- removed R10: 240, HOSS:0207/7
- removed REG_ADJ: 5k, HOSS:RJ6S
- removed R_CURR: 0.2, HOSS:IMEAS_R
- added C14, R1: ??, cyclops:0603
- added R5: 1k 0.1%, cyclops:0603
- added R6: 0.2, cyclops:2512
- added U1: ADR03AKSZ-REEL7, cyclops:SOT65P210X110-5N
- C4: value 0.1uF -> 1uF; device rcl:C050-024X044 -> cyclops:0805
- C5: value 1.0uF -> 0.1uF; device rcl:C025-024X044 -> cyclops:0603
- C8: device cyclops:0805 -> cyclops:0603
- C9: device cyclops:0603 -> cyclops:0805
- IC5: device linear:SO14 -> cyclops:SO14
- R12, R9: device HOSS:0207/7 -> cyclops:0603
- R2: value 1.5k -> 4k 0.1%; device HOSS:0207/7 -> cyclops:0603
- moved C7 257.8 mm to (239.7, -10.2)
- moved CTL_K 257.8 mm to (372.4, 9.21)
- moved CURR/OPT 257.8 mm to (355.3, -47.9)
- moved JP2 257.8 mm to (281.3, -106.7)
- moved JP4 257.8 mm to (285.4, -89.2)
- moved R3 257.8 mm to (235.9, -32.4)
- moved R4 257.8 mm to (241.6, -23.5)
- moved R9 257.8 mm to (237.5, -52.1)
- moved TEST 257.8 mm to (336.9, -40.3)
- moved C2 257.8 mm to (240.3, -16.5)
- moved C3 257.8 mm to (221.0, -58.4)
- moved JP3 257.8 mm to (286.4, -82.9)
- moved JP5 257.8 mm to (282.9, -95.9)
- moved JP6 257.8 mm to (366.1, -7.62)
- moved R12 257.8 mm to (238.1, -3.49)
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Connections:
- removed net N$14: IC5.10, JP1.2
- removed net N$17: JP1.5, JP1.6
- removed net N$18: JP1.3
- removed net N$24: R9.1, REF_ADJ.A
- removed net N$28: ON.A, R2.1
- removed net P_SUP: C4.1, IC2.S
- new net TEMP: U1.1
- net +12V: now also C4.1, C5.1, U1.3
- net CS0: now also S1.5, U$2.D0; no longer S1.8, U$2.D1
- net CS1: now also S1.6, U$2.D1; no longer S1.7, U$2.D2
- net CS2: now also S1.7, U$2.D2; no longer S1.6, U$2.D3
- net CS3: now also S1.8, U$2.D3; no longer S1.5, U$2.D4
- net DACA: now also C14.1, R1.2
- net GND: now also C14.2, R1.1, R5.2, R6.1, R9.1, U1.2; no longer C6.2, GND2.P$1, IC3.4, IMEAS_K.A, ON.K, R9.2, REG_ADJ.S, R_CURR.1
- net LDAC: now also U$2.D4; no longer U$2.D0
- net N$15: now also R2.1; no longer IMEAS_K.S
- net N$19: now also R9.2, REF_ADJ.E; no longer IC2.G, R10.1, REG_ADJ.E
- net N$2: now also R6.2; no longer R_CURR.2
- net N$20: now also U1.5; no longer IC3.5
- net N$4: now also R2.2, R5.1; no longer IMEAS_K.E
- net N$8: now also IC5.10; no longer JP1.4
- net N$9: no longer IC5.8, JP1.1
- net P_12V: no longer +12V.P$1, C5.1, C6.1, IC2.D, IC3.2, R10.2, R2.2
- net REFA: now also REF_ADJ.A, U1.4
- net REF_5V: no longer IC3.6, REF_ADJ.E
Routing:
- net GND: track 76.4 -> 0.00 mm
- net N$2: track 39.2 -> 0.00 mm
- added copper zone on layer 16, net GND

Commit message: Added reverse polarity protection to power input.
Parts:
- added D3: MMSZ5240B, cyclops:SOD123
- added Q1: SUM11006, transistor-fet:TO220
- added R10: 10k, cyclops:0603
- REF_ADJ: device HOSS:RJ6S -> cyclops:SM-42/43W
- moved REF_ADJ 212.3 mm to (54.0, 19.7)
Connections:
- new net N$14: IC5.13, IC5.14, IC5.3
- new net N$17: POWER.P$1, Q1.2
- new net N$18: D3.A, Q1.1, R10.2
- net +15V: now also D3.C, Q1.3; no longer POWER.P$1
- net GND: now also R10.1
- net N$19: now also REF_ADJ.3; no longer REF_ADJ.E
- net N$22: now also REF_ADJ.2; no longer REF_ADJ.S
- net N$8: now also IC5.12; no longer IC5.3
- net N$9: now also IC5.8
- net REFA: now also REF_ADJ.1; no longer REF_ADJ.A
Changed lines of the file:
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@@
 <attribute name="VALUE" x="371.4115" y="8.3439" size="1.27" layer="27" ratio="10" rot="R90"/>
 </element>
-<element name="REF_ADJ" library="HOSS" package="RJ6S" value="10k" x="266.065" y="9.525" smashed="yes" rot="R270">
-<attribute name="NAME" x="261.112" y="13.335" size="1.27" layer="25" ratio="10" rot="R270"/>
-<attribute name="VALUE" x="267.081" y="11.0236" size="1.27" layer="27" ratio="10" rot="R270"/>
+<element name="REF_ADJ" library="cyclops" package="SM-42/43W" value="10k" x="53.975" y="19.685" smashed="yes" rot="R270">
+<attribute name="NAME" x="49.022" y="23.495" size="1.27" layer="25" ratio="10" rot="R270"/>
+<attribute name="VALUE" x="54.991" y="21.1836" size="1.27" layer="27" ratio="10" rot="R270"/>
 </element>
 <element name="R9" library="cyclops" package="0603" value="1k" x="237.49" y="-52.07" rot="R90">
@@
 </element>
 <element name="C5" library="cyclops" package="0603" value="0.1uF" x="35.56" y="41.91" rot="R90"/>
+<element name="Q1" library="transistor-fet" package="TO220" value="SUM11006" x="-7.62" y="-101.6"/>
+<element name="R10" library="cyclops" package="0603" value="10k" x="-6.35" y="-111.76">
+<attribute name="MN" value="Panasonic" x="-6.35" y="-111.76" size="1.778" layer="27" display="off"/>
+<attribute name="DK" value="PxxxxHTR-ND" x="-6.35" y="-111.76" size="1.778" layer="27" display="off"/>
+<attribute name="MPN" value="ERJ-3EKFxxxxV" x="-6.35" y="-111.76" size="1.778" layer="27" display="off"/>
+</element>
+<element name="D3" library="cyclops" package="SOD123" value="MMSZ5240B" x="-8.89" y="-116.84"/>
 </elements>
 <signals>
@@
 </signal>
 <signal name="N$8">
-<contactref element="IC5" pad="3"/>
 <contactref element="CTL_K" pad="S"/>
 <contactref element="IC5" pad="10"/>
-<wire x1="33.9725" y1="26.61" x2="375.1675" y2="9.2075" width="0" layer="19" extent="1-1"/>
-<wire x1="36.5125" y1="31.81" x2="33.9725" y2="26.61" width="0" layer="19" extent="1-1"/>
+<contactref element="IC5" pad="12"/>
+<wire x1="36.5125" y1="31.81" x2="375.1675" y2="9.2075" width="0" layer="19" extent="1-1"/>
+<wire x1="33.9725" y1="31.81" x2="36.5125" y2="31.81" width="0" layer="19" extent="1-1"/>
 </signal>
 <signal name="N$11">
@@
 <signal name="N$9">
 <contactref element="IC5" pad="9"/>
+<contactref element="IC5" pad="8"/>
+<wire x1="37.7825" y1="31.81" x2="39.0525" y2="31.81" width="0" layer="19" extent="1-1"/>
 </signal>
 <signal name="N$12">
@@
 <signal name="N$22">
 <contactref element="R12" pad="1"/>
-<contactref element="REF_ADJ" pad="S"/>
-<wire x1="263.325" y1="9.525" x2="237.2614" y2="-3.4925" width="0" layer="19" extent="1-1"/>
+<contactref element="REF_ADJ" pad="2"/>
+<wire x1="55.425" y1="19.685" x2="237.2614" y2="-3.4925" width="0" layer="19" extent="1-1"/>
 </signal>
 <signal name="N$27">
@@
 <contactref element="C4" pad="2"/>
 <contactref element="C5" pad="2"/>
+<contactref element="R10" pad="1"/>
 <wire x1="238.76" y1="-44.45" x2="237.1725" y2="-10.16" width="0" layer="19" extent="1-1"/>
 <wire x1="237.49" y1="-52.9336" x2="238.76" y2="-44.45" width="0" layer="19" extent="1-1"/>
@@
 <wire x1="282.575" y1="-106.68" x2="286.7025" y2="-89.2175" width="0" layer="19" extent="1-1"/>
 <wire x1="350.8375" y1="-3.81" x2="286.7025" y2="-89.2175" width="0" layer="19" extent="1-1"/>
+<wire x1="350.8375" y1="-1.27" x2="350.8375" y2="-3.81" width="0" layer="19" extent="1-1"/>
+<wire x1="350.8375" y1="1.27" x2="350.8375" y2="-1.27" width="0" layer="19" extent="1-1"/>
+<wire x1="350.8375" y1="3.81" x2="350.8375" y2="1.27" width="0" layer="19" extent="1-1"/>
+<wire x1="350.8375" y1="6.35" x2="350.8375" y2="3.81" width="0" layer="19" extent="1-1"/>
+<wire x1="350.8375" y1="8.89" x2="350.8375" y2="6.35" width="0" layer="19" extent="1-1"/>
 <wire x1="60.7314" y1="21.59" x2="219.71" y2="-58.42" width="0" layer="19" extent="1-1"/>
 <wire x1="60.5536" y1="24.13" x2="60.7314" y2="21.59" width="0" layer="19" extent="1-1"/>
@@
 <wire x1="48.26" y1="24.5364" x2="49.53" y2="28.1686" width="0" layer="19" extent="1-1"/>
 <wire x1="45.72" y1="24.5364" x2="48.26" y2="24.5364" width="0" layer="19" extent="1-1"/>
+<wire x1="35.2425" y1="31.81" x2="45.72" y2="24.5364" width="0" layer="19" extent="1-1"/>
+<wire x1="35.56" y1="42.7736" x2="35.2425" y2="31.81" width="0" layer="19" extent="1-1"/>
+<wire x1="38.1" y1="42.9514" x2="35.56" y2="42.7736" width="0" layer="19" extent="1-1"/>
+<wire x1="40.8686" y1="41.91" x2="38.1" y2="42.9514" width="0" layer="19" extent="1-1"/>
+<wire x1="26.7335" y1="50.8" x2="35.56" y2="42.7736" width="0" layer="19" extent="1-1"/>
 <wire x1="48.895" y1="10.0965" x2="48.26" y2="24.5364" width="0" layer="19" extent="1-1"/>
 <wire x1="41.5925" y1="9.65" x2="48.895" y2="10.0965" width="0" layer="19" extent="1-1"/>
@@
 <wire x1="24.1935" y1="7.62" x2="30.7086" y2="9.2075" width="0" layer="19" extent="1-1"/>
 <wire x1="23.8125" y1="2.8575" x2="24.1935" y2="7.62" width="0" layer="19" extent="1-1"/>
-<wire x1="35.2425" y1="31.81" x2="26.7335" y2="50.8" width="0" layer="19" extent="1-1"/>
+<wire x1="40.9575" y1="2.54" x2="41.5925" y2="9.65" width="0" layer="19" extent="1-1"/>
 <wire x1="11.395" y1="40.64" x2="26.7335" y2="50.8" width="0" layer="19" extent="1-1"/>
 <wire x1="14.8336" y1="27.94" x2="11.395" y2="40.64" width="0" layer="19" extent="1-1"/>
-<wire x1="40.8686" y1="41.91" x2="23.8125" y2="2.8575" width="0" layer="19" extent="1-1"/>
-<wire x1="38.1" y1="42.9514" x2="40.8686" y2="41.91" width="0" layer="19" extent="1-1"/>
-<wire x1="35.56" y1="42.7736" x2="38.1" y2="42.9514" width="0" layer="19" extent="1-1"/>
+<wire x1="-7.2136" y1="-111.76" x2="23.8125" y2="2.8575" width="0" layer="19" extent="1-1"/>
 </signal>
 <signal name="N$6">
@@
 <contactref element="IC1" pad="3"/>
 <contactref element="D1" pad="C"/>
-<contactref element="POWER" pad="P$1"/>
 <contactref element="C10" pad="+"/>
-<wire x1="23.6982" y1="16.1925" x2="24.67" y2="20.0025" width="0" layer="19" extent="1-1"/>
-<wire x1="20.8915" y1="7.62" x2="23.6982" y2="16.1925" width="0" layer="19" extent="1-1"/>
-<wire x1="21.2725" y1="2.8575" x2="20.8915" y2="7.62" width="0" layer="19" extent="1-1"/>
+<contactref element="Q1" pad="3"/>
+<contactref element="D3" pad="C"/>
+<wire x1="-5.08" y1="-107.95" x2="-7.2516875" y2="-116.84" width="0" layer="19" extent="1-1"/>
+<wire x1="20.8915" y1="7.62" x2="-5.08" y2="-107.95" width="0" layer="19" extent="1-1"/>
+<wire x1="23.6982" y1="16.1925" x2="20.8915" y2="7.62" width="0" layer="19" extent="1-1"/>
+<wire x1="24.67" y1="20.0025" x2="23.6982" y2="16.1925" width="0" layer="19" extent="1-1"/>
 </signal>
 <signal name="+12V">
@@
 <contactref element="C1" pad="1"/>
 <contactref element="U1" pad="4"/>
-<contactref element="REF_ADJ" pad="A"/>
+<contactref element="REF_ADJ" pad="1"/>
 <wire x1="53.28" y1="28.575" x2="42.9514" y2="41.2496" width="0" layer="19" extent="1-1"/>
 <wire x1="49.53" y1="30.2514" x2="53.28" y2="28.575" width="0" layer="19" extent="1-1"/>
-<wire x1="265.865" y1="6.985" x2="53.28" y2="28.575" width="0" layer="19" extent="1-1"/>
+<wire x1="52.525" y1="20.955" x2="53.28" y2="28.575" width="0" layer="19" extent="1-1"/>
 </signal>
 <signal name="DACA">
@@
 </signal>
 <signal name="N$19">
-<contactref element="REF_ADJ" pad="E"/>
+<contactref element="REF_ADJ" pad="3"/>
 <contactref element="R9" pad="2"/>
-<wire x1="265.865" y1="12.065" x2="237.49" y2="-51.2064" width="0" layer="19" extent="1-1"/>
+<wire x1="52.525" y1="18.415" x2="237.49" y2="-51.2064" width="0" layer="19" extent="1-1"/>
+</signal>
+<signal name="N$14">
+<contactref element="IC5" pad="13"/>
+<contactref element="IC5" pad="14"/>
+<contactref element="IC5" pad="3"/>
+<wire x1="31.4325" y1="31.81" x2="32.7025" y2="31.81" width="0" layer="19" extent="1-1"/>
+<wire x1="33.9725" y1="26.61" x2="32.7025" y2="31.81" width="0" layer="19" extent="1-1"/>
+</signal>
+<signal name="N$17">
+<contactref element="POWER" pad="P$1"/>
+<contactref element="Q1" pad="2"/>
+<wire x1="21.2725" y1="2.8575" x2="-7.62" y2="-107.95" width="0" layer="19" extent="1-1"/>
+</signal>
+<signal name="N$18">
+<contactref element="Q1" pad="1"/>
+<contactref element="R10" pad="2"/>
+<contactref element="D3" pad="A"/>
+<wire x1="-5.4864" y1="-111.76" x2="-10.5283" y2="-116.84" width="0" layer="19" extent="1-1"/>
+<wire x1="-10.16" y1="-107.95" x2="-5.4864" y2="-111.76" width="0" layer="19" extent="1-1"/>
 </signal>
 </signals>

Commit message: Some additions/changes to the schematic. All the power comonents should occupy the bottom of the board. The Heat sink will be on top. Ample via connected the two sides. Mica insert will be needed to insulate the heatsink.
Parts:
- removed C7: 0.1uF, rcl:C050-024X044
- removed POWER: SCREW2, cyclops:SCREW2
- removed TEST: (no value), HOSS:320-938
- removed TP_5V: TPPAD1-13, testpad:P1-13
- added I/O_BLOCK: SCREW8, cyclops:SCREW8
- Q1: device transistor-fet:TO220 -> cyclops:TO-262_01
- moved D3 136.1 mm to (24.1, 15.2), turned to 180 degrees
- moved R10 128.1 mm to (24.1, 12.7), turned to 180 degrees
- moved Q1 117.3 mm to (12.7, 14.0), flipped to the bottom, turned to 270 degrees
- moved C10 19.1 mm to (23.8, 26.7)
- moved IC1 13.6 mm to (10.2, 25.7), flipped to the bottom, turned to 270 degrees
Connections:
- removed net N$23: TEST.P$3, TEST.P$5
- removed net P_12V: C7.1, IC5.4
- removed net REF_5V: TEST.P$1, TEST.P$6, TP_5V.TP
- new net BUFTEMP: I/O_BLOCK.P$8
- new net LED+: I/O_BLOCK.P$3
- new net LED-: I/O_BLOCK.P$4
- new net N$21: JP2.3, R5.2, R6.1
- new net V+: IC5.4
- new net V-: IC5.11
- new net VAUX: I/O_BLOCK.P$7
- new net VI: I/O_BLOCK.P$6
- new net VREF: I/O_BLOCK.P$5
- net +15V: now also Q1.S; no longer Q1.3
- net GND: now also I/O_BLOCK.P$2; no longer C7.2, IC5.11, JP2.3, POWER.P$2, R5.2, R6.1
- net N$10: now also I/O_BLOCK.P$1; no longer TEST.P$4
- net N$17: now also Q1.D; no longer POWER.P$1, Q1.2
- net N$18: now also Q1.G; no longer Q1.1
- net N$6: no longer TEST.P$2

Commit message: Added phase-reversal protection circuit to user supplied input pin (which used to go right to the noninverting pin of the LM324.
Parts:
- removed C2: 0.1uF, rcl:C050-024X044
- removed C3: 1uF, rcl:C025-024X044
- removed JP2: (no value), jumper:JP3Q
- removed JP3, JP4, JP5, JP6: (no value), jumper:JP1
- added C15, C17, C7: 1uF, cyclops:0805
- added C16, C18, C6: 0.1uF, cyclops:0603
- added D4, D5: 1N4148WS, cyclops:SOD-323F
- added R13: 10k, cyclops:0603
- added SJ1: (no value), jumper:SJ
- added U2: OP1177, cyclops:SOP65P490X110-8N
- D1, D2: device cyclops:SMA-DO214AC -> cyclops:SMA-DO214AC@1
- DAC: value MCP4921SOIC -> MCP4921
- IC5: value LM324D -> LM324
- R12: value 470 -> 1k
- R2: value 4k 0.1% -> 9k 0.1%
- R3: value 10k -> 470; device HOSS:0207/7 -> cyclops:0603
- R4: value 10k -> 1k; device HOSS:0207/7 -> cyclops:0603
- R8: value 120 -> 1k; device HOSS:0207/7 -> cyclops:0603
- R9: value 1k -> 120
- RSENSE: value 0.2 -> 0.1
- U1: value ADR03AKSZ-REEL7 -> ADR03
- moved R12 268.9 mm to (-10.2, -106.7)
- moved R4 258.5 mm to (-11.4, -76.2), turned to 0 degrees
- moved CTL_K 257.9 mm to (115.9, 35.9)
- moved CURR/OPT 257.9 mm to (98.7, -21.3)
- moved R8 256.9 mm to (-10.2, -104.1), turned to 0 degrees
- moved R3 250.8 mm to (-11.4, -73.7), turned to 0 degrees
- moved R9 250.3 mm to (-11.4, -78.7), turned to 0 degrees
- moved U1 1.27 mm to (43.2, 41.9)
- moved IC5 0.32 mm to (35.6, 29.2)
- moved U$2 0.32 mm to (0.00, 0.00)
- renumbered R6 to RSENSE
Connections:
- net N$1 renamed VFB
- removed net N$12: CTL_K.A, JP2.6
- removed net N$13: C2.2, R8.2
- removed net N$14: IC5.13, IC5.14, IC5.3
- removed net N$16: JP2.2
- removed net N$21: JP2.3, R5.2, RSENSE.1
- removed net N$27: JP4.2, R3.1
- removed net N$29: JP3.1, JP5.1, JP6.2, R4.1
- removed net N$6: JP2.4
- removed net N$69: JP6.1
- removed net N$8: CTL_K.S, IC5.10, IC5.12
- removed net N$9: IC5.8, IC5.9
- removed net V+: IC5.4
- removed net V-: IC5.11
- net +12V: now also C15.1, C16.1, C17.1, C18.1, IC5.4, R12.1, U2.7
- net BUFTEMP: now also U2.2, U2.6
- net GND: now also C15.2, C16.2, C17.2, C18.2, C7.2, CTL_K.E, D4.C, IC5.11, R13.2, R5.2, RSENSE.1, U2.4; no longer C3.2, JP4.1, R8.1
- net N$11: now also C6.1, C7.1, SJ1.2; no longer C2.1, C3.1, JP5.2, R3.2
- net N$19: no longer R9.2
- net N$20: now also R3.2; no longer R12.2
- net N$22: now also R3.1; no longer R12.1
- net N$3: now also SJ1.1; no longer JP3.2, R4.2
- net N$4: now also C6.2, R9.2; no longer CURR/OPT.P$1, IC5.7, R2.2, R5.1
- net N$5: now also D4.A, R12.2, R8.2; no longer CURR/OPT.P$3
- net N$7: now also CTL_K.S, D5.A, R8.1; no longer CTL_K.E, JP2.5
- net TEMP: now also U2.3
- net VAUX: now also CURR/OPT.P$3
- net VI: now also CURR/OPT.P$1, IC5.7, R2.2, R5.1
- net VIN: now also CTL_K.A
- net VREF: now also D5.C, IC5.10, IC5.3, IC5.8, IC5.9, R13.1
Routing:
- removed copper zone on layer 1, net GND
Other:
- board size 132.2 x 81.4 mm -> 68.6 x 53.3 mm
- board text removed: "+"
- board text removed: "1 W 3"
- board text removed: "LED+ LED- 12V GND"
- board text removed: "VIN GND"
- board text removed: "VPD VI VR VC GND"
