File: pcb/cyclops_r3/cyclops_r3p1.brd (EAGLE design)
At the start: 69.8 x 53.3 mm, 48 parts, among them Q1 SUM11006, Q2 IRF510, U1 MCP4921, U2 317-N, U3 ADR03, U4 OP1177, U5 LM324N, U6 ZXTD45

Commit message: Minor changes.
Routing:
- net GND: track 65.8 -> 67.9 mm
Changed lines of the file:
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@@
 </plain>
 <attributes>
+<attribute name="PCB" value="Cyclops r3.1"/>
+<attribute name="REVISION" value="3.1"/>
 </attributes>
 <variantdefs>
@@
 </element>
 <element name="D2" library="cyclops" package="SMA-DO214AC" value="S1B" x="44.196" y="9.144" smashed="yes" rot="R270">
-<attribute name="NAME" x="42.418" y="5.588" size="0.889" layer="25" font="vector" ratio="18" rot="R90"/>
-<attribute name="VALUE" x="42.418" y="7.366" size="0.889" layer="27" font="vector" ratio="18" rot="R90"/>
+<attribute name="NAME" x="42.418" y="6.096" size="0.889" layer="25" font="vector" ratio="18" rot="R90"/>
+<attribute name="VALUE" x="42.418" y="8.128" size="0.889" layer="27" font="vector" ratio="18" rot="R90"/>
 </element>
 <element name="R3" library="cyclops" package="0603" value="1.8k" x="45.72" y="16.002" smashed="yes" rot="R90">
@@
 </element>
 <element name="C5" library="cyclops" package="1206-POL" value="1uF" x="40.132" y="8.128" smashed="yes" rot="R270">
-<attribute name="NAME" x="38.608" y="5.588" size="0.889" layer="25" font="vector" ratio="18" rot="R90"/>
-<attribute name="VALUE" x="38.608" y="7.62" size="0.889" layer="27" font="vector" ratio="18" rot="R90"/>
+<attribute name="NAME" x="38.608" y="6.096" size="0.889" layer="25" font="vector" ratio="18" rot="R90"/>
+<attribute name="VALUE" x="38.608" y="8.128" size="0.889" layer="27" font="vector" ratio="18" rot="R90"/>
 </element>
 <element name="C6" library="cyclops" package="1206-POL" value="10uF" x="48.26" y="8.128" smashed="yes" rot="R270">
-<attribute name="NAME" x="46.736" y="5.588" size="0.889" layer="25" font="vector" ratio="18" rot="R90"/>
-<attribute name="VALUE" x="46.736" y="7.62" size="0.889" layer="27" font="vector" ratio="18" rot="R90"/>
+<attribute name="NAME" x="46.736" y="6.096" size="0.889" layer="25" font="vector" ratio="18" rot="R90"/>
+<attribute name="VALUE" x="46.736" y="8.128" size="0.889" layer="27" font="vector" ratio="18" rot="R90"/>
 </element>
 <element name="C9" library="cyclops" package="1206-POL" value="1uF" x="54.356" y="25.908" smashed="yes">
@@
 <wire x1="58.168" y1="9.146" x2="58.168" y2="9.906" width="1.27" layer="1"/>
 <via x="41.91" y="13.716" extent="1-16" drill="1" shape="octagon"/>
-<via x="40.132" y="4.826" extent="1-16" drill="1" shape="octagon"/>
-<via x="48.26" y="4.826" extent="1-16" drill="1" shape="octagon"/>
-<wire x1="40.132" y1="4.826" x2="40.132" y2="6.477" width="0.8128" layer="1"/>
-<wire x1="48.26" y1="4.826" x2="48.26" y2="6.477" width="0.8128" layer="1"/>
+<via x="41.91" y="5.334" extent="1-16" drill="1" shape="octagon"/>
+<via x="50.292" y="5.334" extent="1-16" drill="1" shape="octagon"/>
+<wire x1="41.91" y1="5.334" x2="40.699959375" y2="5.334" width="0.8128" layer="1"/>
+<wire x1="40.699959375" y1="5.334" x2="40.132" y2="5.901959375" width="0.8128" layer="1"/>
+<wire x1="40.132" y1="5.901959375" x2="40.132" y2="6.477" width="0.8128" layer="1"/>
+<wire x1="50.292" y1="5.334" x2="48.827959375" y2="5.334" width="0.8128" layer="1"/>
+<wire x1="48.827959375" y1="5.334" x2="48.26" y2="5.901959375" width="0.8128" layer="1"/>
+<wire x1="48.26" y1="5.901959375" x2="48.26" y2="6.477" width="0.8128" layer="1"/>
 <wire x1="45.72" y1="15.1384" x2="43.18" y2="15.1384" width="0.8128" layer="1"/>
 <wire x1="43.18" y1="15.1384" x2="42.56055625" y2="15.1384" width="0.8128" layer="1"/>
@@
 <wire x1="15.494" y1="25.4" x2="14.628" y2="25.4" width="0.6096" layer="16"/>
 <wire x1="14.628" y1="25.4" x2="14.562" y2="25.466" width="0.6096" layer="16"/>
-<wire x1="12.7" y1="23.2156" x2="12.7" y2="23.876" width="0.6096" layer="16"/>
-<wire x1="12.7" y1="23.876" x2="13.462" y2="24.638" width="0.6096" layer="16"/>
-<wire x1="13.462" y1="24.638" x2="13.734" y2="24.638" width="0.6096" layer="16"/>
-<wire x1="13.734" y1="24.638" x2="14.562" y2="25.466" width="0.6096" layer="16"/>
+<wire x1="14.562" y1="25.466" x2="12.7" y2="23.604" width="0.6096" layer="16"/>
+<wire x1="12.7" y1="23.604" x2="12.7" y2="23.2156" width="0.6096" layer="16"/>
 </signal>
 <signal name="N$13">

Commit message: Minor changes.
Parts:
- removed R14: 560, cyclops:0603
- added R12: 560, cyclops:0603
- R10: value 1.1k -> 560
- R11: value 560 -> 1.1k
- moved R10 4.79 mm to (12.7, 22.4), turned to 270 degrees
- moved R11 1.78 mm to (10.2, 26.4), turned to 90 degrees
- renumbered C16 to C15
Connections:
- net +12V: now also R11.2; no longer R10.2
- net GND: now also R12.1; no longer R11.1
- net N$10: now also R10.1; no longer R14.1
- net N$13: now also R10.2, R11.1, R12.2; no longer R10.1, R11.2, R14.2
Changed lines of the file:
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@@
 <setting verticaltext="up"/>
 </settings>
-<grid distance="0.01" unitdist="inch" unit="inch" style="lines" multiple="1" display="yes" altdistance="0.025" altunitdist="inch" altunit="inch"/>
+<grid distance="0.005" unitdist="inch" unit="inch" style="lines" multiple="1" display="yes" altdistance="0.025" altunitdist="inch" altunit="inch"/>
 <layers>
 <layer number="1" name="Top" color="4" fill="1" visible="yes" active="yes"/>
@@
 <layer number="27" name="tValues" color="7" fill="1" visible="yes" active="yes"/>
 <layer number="28" name="bValues" color="7" fill="1" visible="yes" active="yes"/>
-<layer number="29" name="tStop" color="7" fill="3" visible="no" active="yes"/>
+<layer number="29" name="tStop" color="7" fill="3" visible="yes" active="yes"/>
 <layer number="30" name="bStop" color="7" fill="6" visible="no" active="yes"/>
 <layer number="31" name="tCream" color="7" fill="4" visible="no" active="yes"/>
@@
 <attribute name="VALUE" x="44.45" y="35.56" size="0.889" layer="27" font="vector" ratio="18"/>
 </element>
-<element name="C16" library="cyclops" package="0805" value="1uF" x="19.304" y="45.212" smashed="yes" rot="R270">
+<element name="C15" library="cyclops" package="0805" value="1uF" x="19.304" y="45.212" smashed="yes" rot="R270">
 <attribute name="MN" value="TDK Corp." x="19.304" y="45.212" size="1.778" layer="27" rot="R270" display="off"/>
 <attribute name="PARTNO" value="C2012X5R1Cxxxxxxx" x="19.304" y="45.212" size="1.778" layer="27" rot="R270" display="off"/>
@@
 </element>
 <element name="S3" library="cyclops" package="CFPA" value="TEST" x="3.81" y="47.244" smashed="yes">
-<attribute name="NAME" x="2.54" y="46.736" size="0.889" layer="25" font="vector" ratio="18" rot="R90"/>
-<attribute name="VALUE" x="5.842" y="45.974" size="0.889" layer="27" font="vector" ratio="18" rot="R90"/>
+<attribute name="NAME" x="5.461" y="46.736" size="0.889" layer="25" font="vector" ratio="18" rot="R90"/>
+<attribute name="VALUE" x="6.604" y="45.974" size="0.889" layer="27" font="vector" ratio="18" rot="R90"/>
 </element>
 <element name="U6" library="cyclops" package="SOT23-6" value="ZXTD45" x="13.462" y="26.416" smashed="yes" rot="MR90">
@@
 <attribute name="VALUE" x="5.842" y="11.176" size="0.889" layer="28" font="vector" ratio="18" rot="MR90"/>
 </element>
-<element name="R14" library="cyclops" package="0603" value="560" x="12.7" y="22.352" smashed="yes" rot="MR270">
+<element name="R10" library="cyclops" package="0603" value="560" x="12.7" y="22.352" smashed="yes" rot="MR270">
 <attribute name="MN" value="Panasonic" x="12.7" y="22.352" size="1.778" layer="28" rot="MR270" display="off"/>
 <attribute name="DK" value="PxxxxHTR-ND" x="12.7" y="22.352" size="1.778" layer="28" rot="MR270" display="off"/>
@@
 <attribute name="VALUE" x="13.716" y="18.542" size="0.889" layer="28" font="vector" ratio="18" rot="MR0"/>
 </element>
-<element name="R10" library="cyclops" package="0603" value="1.1k" x="10.16" y="26.416" smashed="yes" rot="MR90">
+<element name="R11" library="cyclops" package="0603" value="1.1k" x="10.16" y="26.416" smashed="yes" rot="MR90">
 <attribute name="MN" value="Panasonic" x="10.16" y="26.416" size="0.889" layer="28" ratio="15" rot="MR90" display="off"/>
 <attribute name="DK" value="PxxxxHTR-ND" x="10.16" y="26.416" size="0.889" layer="28" ratio="15" rot="MR90" display="off"/>
@@
 <attribute name="VALUE" x="8.636" y="20.828" size="0.889" layer="28" font="vector" ratio="18" rot="MR0" align="center-left"/>
 </element>
-<element name="R11" library="cyclops" package="0603" value="560" x="8.382" y="26.416" smashed="yes" rot="MR270">
+<element name="R12" library="cyclops" package="0603" value="560" x="8.382" y="26.416" smashed="yes" rot="MR270">
 <attribute name="MN" value="Panasonic" x="8.382" y="26.416" size="0.889" layer="28" ratio="15" rot="MR270" display="off"/>
 <attribute name="DK" value="PxxxxHTR-ND" x="8.382" y="26.416" size="0.889" layer="28" ratio="15" rot="MR270" display="off"/>
@@
 <wire x1="67.564" y1="31.242" x2="66.548" y2="32.258" width="0.3048" layer="1"/>
 <wire x1="66.548" y1="32.258" x2="64.77" y2="32.258" width="0.3048" layer="1"/>
-<wire x1="64.77" y1="32.258" x2="63.754" y2="33.274" width="0.3048" layer="1"/>
-<wire x1="63.754" y1="33.274" x2="63.754" y2="35.814" width="0.3048" layer="1"/>
-<wire x1="63.754" y1="35.814" x2="62.865" y2="36.703" width="0.3048" layer="1"/>
+<wire x1="64.77" y1="32.258" x2="63.627" y2="33.401" width="0.3048" layer="1"/>
+<wire x1="63.627" y1="33.401" x2="63.627" y2="35.941" width="0.3048" layer="1"/>
+<wire x1="63.627" y1="35.941" x2="62.865" y2="36.703" width="0.3048" layer="1"/>
 <wire x1="62.865" y1="36.703" x2="61.528" y2="36.703" width="0.3048" layer="1"/>
 </signal>
@@
 <contactref element="U4" pad="7"/>
 <contactref element="C14" pad="1"/>
-<contactref element="C16" pad="1"/>
+<contactref element="C15" pad="1"/>
 <contactref element="D3" pad="C"/>
 <contactref element="I/O_BLOCK" pad="P$3"/>
@@
 <via x="21.082" y="23.876" extent="1-16" drill="0.3302"/>
 <via x="20.066" y="23.876" extent="1-16" drill="0.3302"/>
-<contactref element="R10" pad="2"/>
+<contactref element="R11" pad="2"/>
 <contactref element="U6" pad="1"/>
 <wire x1="10.16" y1="27.2796" x2="10.5664" y2="27.2796" width="0.6096" layer="16"/>
@@
 <wire x1="35.306" y1="19.05" x2="38.354" y2="16.002" width="0.4064" layer="16"/>
 <wire x1="38.354" y1="16.002" x2="38.354" y2="7.317803125" width="0.4064" layer="16"/>
-<wire x1="38.354" y1="7.317803125" x2="35.862196875" y2="4.826" width="0.4064" layer="16"/>
-<wire x1="35.862196875" y1="4.826" x2="29.21" y2="4.826" width="0.4064" layer="16"/>
-<wire x1="29.21" y1="4.826" x2="6.503809375" y2="4.826" width="0.4064" layer="1"/>
-<wire x1="6.503809375" y1="4.826" x2="5.588" y2="5.741809375" width="0.4064" layer="1"/>
+<wire x1="38.354" y1="7.317803125" x2="36.116196875" y2="5.08" width="0.4064" layer="16"/>
+<wire x1="36.116196875" y1="5.08" x2="29.21" y2="5.08" width="0.4064" layer="16"/>
+<wire x1="29.21" y1="5.08" x2="6.249809375" y2="5.08" width="0.4064" layer="1"/>
+<wire x1="6.249809375" y1="5.08" x2="5.588" y2="5.741809375" width="0.4064" layer="1"/>
 <wire x1="5.588" y1="5.741809375" x2="5.588" y2="10.414" width="0.4064" layer="1"/>
 <wire x1="5.588" y1="10.414" x2="3.556" y2="12.446" width="0.4064" layer="1"/>
 <wire x1="45.6438" y1="26.5938" x2="45.974" y2="26.924" width="0.4064" layer="1"/>
 <wire x1="45.974" y1="26.924" x2="46.3042" y2="27.2542" width="0.4064" layer="1"/>
-<via x="29.21" y="4.826" extent="1-16" drill="0.5"/>
+<via x="29.21" y="5.08" extent="1-16" drill="0.5"/>
 </signal>
 <signal name="VCTL">
@@
 <contactref element="RSENSE" pad="1"/>
 <contactref element="U4" pad="4"/>
-<contactref element="C16" pad="2"/>
+<contactref element="C15" pad="2"/>
 <contactref element="C14" pad="2"/>
 <contactref element="D4" pad="A"/>
@@
 <contactref element="U$1" pad="GND$1"/>
 <contactref element="U$1" pad="GND"/>
-<contactref element="R11" pad="1"/>
+<contactref element="R12" pad="1"/>
 <via x="6.858" y="27.178" extent="1-16" drill="0.5"/>
 <wire x1="8.382" y1="27.2796" x2="8.5344" y2="27.178" width="0.6096" layer="16"/>
@@
 <wire x1="8.89" y1="36.576" x2="4.318" y2="41.148" width="0.4064" layer="1"/>
 <wire x1="4.318" y1="41.148" x2="4.318" y2="43.18" width="0.4064" layer="1"/>
-<wire x1="0.762" y1="46.736" x2="0.762" y2="48.514" width="0.4064" layer="1"/>
-<wire x1="0.762" y1="48.514" x2="1.016" y2="48.768" width="0.4064" layer="1"/>
-<via x="1.016" y="48.768" extent="1-16" drill="0.5"/>
-<wire x1="1.016" y1="48.768" x2="1.016" y2="50.994040625" width="0.4064" layer="16"/>
-<wire x1="1.016" y1="50.994040625" x2="1.583959375" y2="51.562" width="0.4064" layer="16"/>
+<wire x1="0.762" y1="46.736" x2="0.762" y2="48.768" width="0.4064" layer="1"/>
+<via x="0.762" y="48.768" extent="1-16" drill="0.5"/>
+<wire x1="0.762" y1="50.740040625" x2="1.583959375" y2="51.562" width="0.4064" layer="16"/>
 <wire x1="1.583959375" y1="51.562" x2="2.286" y2="51.562" width="0.4064" layer="16"/>
 <wire x1="2.286" y1="51.562" x2="2.794" y2="51.054" width="0.4064" layer="16"/>
@@
 <wire x1="3.556" y1="17.526" x2="8.89" y2="22.86" width="0.4064" layer="1"/>
 <wire x1="0.762" y1="46.736" x2="4.318" y2="43.18" width="0.4064" layer="1"/>
+<wire x1="0.762" y1="50.740040625" x2="0.762" y2="48.768" width="0.4064" layer="16"/>
 </signal>
 <signal name="N$1">
@@
 <contactref element="U6" pad="6"/>
 <contactref element="U6" pad="4"/>
-<contactref element="R14" pad="1"/>
+<contactref element="R10" pad="1"/>
 <wire x1="14.562" y1="27.366" x2="15.43199375" y2="27.366" width="0.6096" layer="16"/>
 <wire x1="15.43199375" y1="27.366" x2="15.748" y2="27.04999375" width="0.6096" layer="16"/>
@@
 <signal name="N$13">
 <contactref element="Q2" pad="G"/>
-<contactref element="R14" pad="2"/>
+<contactref element="R10" pad="2"/>
 <wire x1="12.7" y1="21.4884" x2="10.3124" y2="21.4884" width="0.6096" layer="16"/>
 <wire x1="10.3124" y1="21.4884" x2="10.16" y2="21.336" width="0.4064" layer="16"/>
 <wire x1="10.16" y1="21.336" x2="10.16" y2="22.3647" width="0.4064" layer="16"/>
-<contactref element="R10" pad="1"/>
-<contactref element="R11" pad="2"/>
+<contactref element="R11" pad="1"/>
+<contactref element="R12" pad="2"/>
 <wire x1="10.16" y1="22.3647" x2="10.16" y2="25.5524" width="0.6096" layer="16"/>
 <wire x1="10.16" y1="25.5524" x2="8.382" y2="25.5524" width="0.6096" layer="16"/>
 </signal>
 </signals>
+<errors>
+</errors>
 </board>
 </drawing>
