File: pcb/cyclops_r3/cyclops_r3p1.sch (EAGLE design)
At the start: 74 parts, among them Q1 SUM11006, Q2 IRF510, U1 MCP4921, U2 317-N, U3 ADR03, U4 OP1177, U5 LM324N, U6 ZXTD45, U8 TLV3701CDBVT

Commit message: Added a negative rail, used exclusively by the opamp, to allow a wider bandwidth. Finished routing everything. Need to make bottom silkscreen and finish testing comparitor circuit.
Parts:
- removed 12V: SCREW2, cyclops:SCREW2
- removed R50: 2.4k, cyclops:R_0603
- added C20: 1uF, cyclops:C_0805
- added C21: .1uF, cyclops:C_0603
- added R22: 9k, cyclops:R_0603
- added R23: 10, cyclops:R_0603
- added R24: 1k, cyclops:R_0603
- added U7: LM324N, cyclops:LM324D
- C10: value 1uF -> 47uF; device cyclops:C_0805 -> cyclops:C-POL_0807
- C11: device cyclops:C_0805 -> cyclops:C-POL_1206
- C12, C13: value .1uF -> 1uF; device cyclops:C_0603 -> cyclops:C-POL_1206
- C14: value .1uF -> 1uF; device cyclops:C_0603 -> cyclops:C_0805
- C19: value 10pF -> .1uF
- C5: value 1uF -> 10pF; device cyclops:C-POL_1206 -> cyclops:C_0603
- C6: value 10uF -> .1uF; device cyclops:C-POL_1206 -> cyclops:C_0603
- C7: value 47uF -> 1uF; device cyclops:C-POL_0807 -> cyclops:C-POL_1206
- C8: value 47uF -> 10uF; device cyclops:C-POL_0807 -> cyclops:C-POL_1206
- C9: value 1uF -> 47uF; device cyclops:C-POL_1206 -> cyclops:C-POL_0807
- D1: value MMSZ -> (none); device cyclops:Z-DIODE_MMSZ -> cyclops:DIODESOD-323
- D2: value S1B -> MMSZ; device cyclops:DIODES1B-13-F -> cyclops:Z-DIODE_MMSZ
- D3: value DS11015 -> S1B; device cyclops:S-DIODESOD-123 -> cyclops:DIODES1B-13-F
- D5: value (none) -> DS11015; device cyclops:DIODESOD-323 -> cyclops:S-DIODESOD-123
- R10: value 10 -> 220k
- R11: value 220k -> 3.0k
- R12: value 1k -> 2.4k
- R13: value 1k -> 75
- R14: value 1k -> 120
- R15: value 1k -> 470
- R16: value 100k -> 1k
- R18: value 3.0k -> 1k
- R19: value 4k -> 1k
- R2: value 10k -> 100k
- R20: value 56k -> 1k
- R21: value 91k -> 1k
- R3: value 2.1k -> 56k
- R4: value 240 -> 10k
- R5: value 470 -> 4k
- R6: value 1k -> 91k
- R8: value 1k -> 240
- R9: value 9k -> 2.1k
- S4: value CURR/AUX -> UNKILL; device cyclops:SPDT_PCM12 -> cyclops:SPST_TACT-EVQQ2
- S5: value UNKILL -> CURR/AUX; device cyclops:SPST_TACT-EVQQ2 -> cyclops:SPDT_PCM12
- U2: value 317-N -> TLV37; device cyclops:317_TO263 -> ti-extended:TLV3701CDBVT
- U3: value ADR03 -> 317-N; device cyclops:ADR03AKSZ-REEL7 -> cyclops:317_TO263
- U4: value OP1177 -> 337-N; device cyclops:OP1177ARMZ -> cyclops:337IMP
- U5: value LM324N -> ADR03; device cyclops:LM324D -> cyclops:ADR03AKSZ-REEL7
- U6: value ZXTD45 -> OP1177; device cyclops:ZXTD4591E6 -> cyclops:OP1177ARMZ
- U8: value TLV3701CDBVT -> ZXTD45; device ti-extended:TLV3701CDBVT -> cyclops:ZXTD4591E6
Connections:
- new net -2.1V: C13.-, C19.2, C20.2, R14.1, U4.VO, U7P.V-
- new net -5V: C12.-, I/O_BLOCK.3, U4.VI
- new net N$12: R13.1, R14.2, U4.ADJ
- net +12V: now also C10.+, C11.+, C16.1, C19.1, C20.1, C21.1, D3.A, D4.C, R12.2, R8.2, U3.VO, U5.VIN, U6.V+, U7P.V+, U8.C1; no longer 12V.2, C10.1, C11.1, C12.1, C13.1, C7.+, C8.+, D2.A, D3.C, I/O_BLOCK.3, R4.2, R50.2, U2.VO, U3.VIN, U4.V+, U5P.V+, U6.C1
- net +15V: now also C6.1, R3.1, U2.VCC; no longer C18.1, R20.1, U8.VCC
- net +15V_RECT: now also C7.+, D3.C, U3.VI; no longer C5.+, D1.C, U2.VI
- net COMP+: now also C5.1, R2.1, R6.2, S4.P, S4.P1, U2.IN+; no longer C19.1, R16.1, R21.2, S5.P, S5.P1, U8.IN+
- net GND: now also C10.-, C11.-, C12.+, C13.+, C21.2, C5.2, C6.2, D5.A, R10.1, R16.1, R18.2, R21.2, R24.1, R4.1, R5.2, R9.1, S4.S, S4.S1, U2.GND, U5.GND, U6.V-, U8.C2; no longer 12V.1, C10.2, C11.2, C12.2, C13.2, C19.2, C5.-, C6.-, D4.A, R11.1, R12.1, R19.2, R2.1, R3.1, R6.1, R8.2, S5.S, S5.S1, U3.GND, U4.V-, U5P.V-, U6.C2, U8.GND
- net KILL: now also D1.A, R10.2, R7.1, U2.OUT; no longer D5.A, R17.1, R18.2, U8.OUT
- net N$10: now also R23.1, U8.E1, U8.E2; no longer R10.1, U6.E1, U6.E2
- net N$11: now also R11.1; no longer R18.1
- net N$13: now also R23.2, R24.2; no longer R10.2, R12.2
- net N$15: now also R22.1, U7B.-IN; no longer R9.1, U5B.-IN
- net N$18: now also D1.C, D2.A, R4.2; no longer D1.A, D5.C, R2.2
- net N$2: now also U7B.+IN; no longer U5B.+IN
- net N$20: now also R15.2, U5.TRIM; no longer R5.2, U3.TRIM
- net N$22: now also R15.1; no longer R5.1
- net N$3: now also R12.1; no longer R50.1
- net N$4: now also U7C.OUT, U8.B1, U8.B2; no longer U5C.OUT, U6.B1, U6.B2
- net N$5: now also R3.2, R5.1, U2.IN-; no longer R19.1, R20.2, U8.IN-
- net N$6: now also R16.2; no longer R6.2
- net N$7: now also R19.1; no longer R7.1
- net N$72: now also C8.+, R8.1, R9.2, U3.ADJ; no longer C6.+, R3.2, R4.1, U2.ADJ
- net N$8: now also R17.2, U7A.-IN; no longer R14.2, U5A.-IN
- net N$9: now also R6.1, R7.2; no longer R17.2, R21.1
- net REFA: now also U5.VOUT, U7A.+IN; no longer U3.VOUT, U5A.+IN
- net REFA2X: now also C18.1, R20.2; no longer C16.1, R15.2
- net TEMP: now also U5.TEMP, U6.+IN; no longer U3.TEMP, U4.+IN
- net VAUX: now also S5.3; no longer S4.3
- net VFB: now also S5.2, U7C.-IN; no longer S4.2, U5C.-IN
- net VI: now also R2.2, R21.1, R22.2, S5.1, U7B.OUT; no longer R16.2, R8.1, R9.2, S4.1, U5B.OUT
- net VREF: now also U7D.-IN, U7D.OUT; no longer U5D.-IN, U5D.OUT
- net VREFA2X: now also R17.1, R18.1, R20.1, U7A.OUT; no longer R13.1, R14.1, R15.1, U5A.OUT
- net VTEMP: now also U6.-IN, U6.OUT; no longer U4.-IN, U4.OUT
- net _VREF: now also D4.A, D5.C, R19.2, U7C.+IN, U7D.+IN; no longer D3.A, D4.C, R7.2, U5C.+IN, U5D.+IN
Other:
- note added: "Neg. Regulation"
- note added: "Pos. Regulation"
- note removed: "Regulation"
