File: cyclops_r3/panel/panels.brd (EAGLE design)
At the start: 0 parts

Commit message: Updated OSH design rules. Some work on panels.
Routing:
- added copper zone on layer 16, net S$1
Other:
- board outline added: 133 x 35 mm
Changed lines of the file:
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@@
 <setting verticaltext="up"/>
 </settings>
-<grid distance="0.05" unitdist="inch" unit="inch" style="lines" multiple="1" display="no" altdistance="0.025" altunitdist="inch" altunit="inch"/>
+<grid distance="1" unitdist="mm" unit="mm" style="lines" multiple="1" display="yes" altdistance="0.025" altunitdist="inch" altunit="inch"/>
 <layers>
 <layer number="1" name="Top" color="4" fill="1" visible="yes" active="yes"/>
@@
 <layer number="27" name="tValues" color="7" fill="1" visible="yes" active="yes"/>
 <layer number="28" name="bValues" color="7" fill="1" visible="yes" active="yes"/>
-<layer number="29" name="tStop" color="7" fill="3" visible="no" active="yes"/>
-<layer number="30" name="bStop" color="7" fill="6" visible="no" active="yes"/>
+<layer number="29" name="tStop" color="7" fill="3" visible="yes" active="yes"/>
+<layer number="30" name="bStop" color="7" fill="6" visible="yes" active="yes"/>
 <layer number="31" name="tCream" color="7" fill="4" visible="no" active="yes"/>
 <layer number="32" name="bCream" color="7" fill="5" visible="no" active="yes"/>
@@
 <layer number="43" name="vRestrict" color="2" fill="10" visible="yes" active="yes"/>
 <layer number="44" name="Drills" color="7" fill="1" visible="no" active="yes"/>
-<layer number="45" name="Holes" color="7" fill="1" visible="no" active="yes"/>
+<layer number="45" name="Holes" color="7" fill="1" visible="yes" active="yes"/>
 <layer number="46" name="Milling" color="3" fill="1" visible="no" active="yes"/>
 <layer number="47" name="Measures" color="7" fill="1" visible="no" active="yes"/>
@@
 <board>
 <plain>
+<wire x1="133" y1="32" x2="133" y2="3" width="0" layer="20"/>
+<wire x1="133" y1="3" x2="130" y2="0" width="0" layer="20" curve="-90"/>
+<wire x1="130" y1="0" x2="3" y2="0" width="0" layer="20"/>
+<wire x1="3" y1="0" x2="0" y2="3" width="0" layer="20" curve="-90"/>
+<wire x1="0" y1="3" x2="0" y2="32" width="0" layer="20"/>
+<wire x1="0" y1="32" x2="3" y2="35" width="0" layer="20" curve="-90"/>
+<wire x1="3" y1="35" x2="130" y2="35" width="0" layer="20"/>
+<wire x1="130" y1="35" x2="133" y2="32" width="0" layer="20" curve="-90"/>
+<hole x="6" y="5.3" drill="3.5"/>
+<hole x="127" y="5.3" drill="3.5"/>
+<hole x="6" y="30.3" drill="3.5"/>
+<hole x="127" y="30.3" drill="3.5"/>
+<hole x="17.077" y="14" drill="11.5"/>
+<hole x="32.825" y="14" drill="11.5"/>
+<hole x="99.246" y="20" drill="9.8"/>
+<hole x="118.296" y="20" drill="9.8"/>
+<wire x1="72.284" y1="21.18" x2="72.284" y2="14.92" width="0" layer="20"/>
+<wire x1="72.284" y1="13.65" x2="92.934" y2="13.65" width="0" layer="20"/>
+<wire x1="92.934" y1="14.92" x2="92.934" y2="21.18" width="0" layer="20"/>
+<wire x1="92.934" y1="22.45" x2="72.284" y2="22.45" width="0" layer="20"/>
+<wire x1="42.636" y1="15.375" x2="42.636" y2="17.125" width="0" layer="20"/>
+<wire x1="49.176" y1="15.375" x2="49.176" y2="17.125" width="0" layer="20"/>
+<wire x1="42.636" y1="17.125" x2="49.176" y2="17.125" width="0" layer="20"/>
+<wire x1="42.636" y1="15.375" x2="49.176" y2="15.375" width="0" layer="20"/>
+<wire x1="55.774" y1="13.65" x2="55.774" y2="19.55" width="0" layer="20"/>
+<wire x1="70.074" y1="13.65" x2="70.074" y2="19.55" width="0" layer="20"/>
+<wire x1="60.924" y1="19.55" x2="60.924" y2="23.55" width="0" layer="20"/>
+<wire x1="55.774" y1="19.55" x2="60.924" y2="19.55" width="0" layer="20"/>
+<wire x1="64.924" y1="19.55" x2="64.924" y2="23.55" width="0" layer="20"/>
+<wire x1="55.774" y1="13.65" x2="70.074" y2="13.65" width="0" layer="20"/>
+<wire x1="64.924" y1="19.55" x2="70.074" y2="19.55" width="0" layer="20"/>
+<wire x1="60.924" y1="23.55" x2="64.924" y2="23.55" width="0" layer="20"/>
+<polygon width="0" layer="30">
+<vertex x="0" y="9"/>
+<vertex x="7" y="9" curve="-90"/>
+<vertex x="10" y="6"/>
+<vertex x="10" y="0"/>
+<vertex x="3" y="0" curve="-90"/>
+<vertex x="0" y="3"/>
+</polygon>
+<polygon width="0" layer="30">
+<vertex x="123" y="0"/>
+<vertex x="123" y="6" curve="-90"/>
+<vertex x="126" y="9"/>
+<vertex x="133" y="9"/>
+<vertex x="133" y="3" curve="-90"/>
+<vertex x="130" y="0"/>
+</polygon>
+<polygon width="0" layer="30">
+<vertex x="123" y="35"/>
+<vertex x="123" y="30" curve="90"/>
+<vertex x="126" y="27"/>
+<vertex x="133" y="27"/>
+<vertex x="133" y="32" curve="90"/>
+<vertex x="130" y="35"/>
+</polygon>
+<polygon width="0" layer="30">
+<vertex x="0" y="27"/>
+<vertex x="7" y="27" curve="90"/>
+<vertex x="10" y="30"/>
+<vertex x="10" y="35"/>
+<vertex x="3" y="35" curve="90"/>
+<vertex x="0" y="32"/>
+</polygon>
+<polygon width="0" layer="30">
+<vertex x="3" y="9"/>
+<vertex x="3" y="27"/>
+<vertex x="0" y="27"/>
+<vertex x="0" y="9"/>
+</polygon>
+<polygon width="0" layer="30">
+<vertex x="10" y="3"/>
+<vertex x="123" y="3"/>
+<vertex x="123" y="0"/>
+<vertex x="10" y="0"/>
+</polygon>
+<polygon width="0" layer="30">
+<vertex x="130" y="27"/>
+<vertex x="130" y="9"/>
+<vertex x="133" y="9"/>
+<vertex x="133" y="27"/>
+</polygon>
+<polygon width="0" layer="30">
+<vertex x="10" y="35"/>
+<vertex x="10" y="32"/>
+<vertex x="123" y="32"/>
+<vertex x="123" y="35"/>
+</polygon>
 </plain>
 <attributes>
@@
 </class>
 </classes>
-<designrules name="default">
+<designrules name="ohs-park-2-layer">
 <description language="de">&lt;b&gt;EAGLE Design Rules&lt;/b&gt;
 &lt;p&gt;
@@
 Einstellungen hier und speichern die Design Rules unter
 einem neuen Namen ab.</description>
-<description language="en">&lt;b&gt;EAGLE Design Rules&lt;/b&gt;
+<description language="en">&lt;b&gt;Laen's PCB Order Design Rules&lt;/b&gt;
 &lt;p&gt;
-The default Design Rules have been set to cover
-a wide range of applications. Your particular design
-may have different requirements, so please make the
-necessary adjustments and save your customized
-design rules under a new name.</description>
+Modified: 2014.10.15
+&lt;p&gt;
+2-layer, OSH Park PCB</description>
 <param name="layerSetup" value="(1*16)"/>
-<param name="mtCopper" value="0.035mm 0.035mm 0.035mm 0.035mm 0.035mm 0.035mm 0.035mm 0.035mm 0.035mm 0.035mm 0.035mm 0.035mm 0.035mm 0.035mm 0.035mm 0.035mm"/>
-<param name="mtIsolate" value="1.5mm 0.15mm 0.2mm 0.15mm 0.2mm 0.15mm 0.2mm 0.15mm 0.2mm 0.15mm 0.2mm 0.15mm 0.2mm 0.15mm 0.2mm"/>
-<param name="mdWireWire" value="8mil"/>
-<param name="mdWirePad" value="8mil"/>
-<param name="mdWireVia" value="8mil"/>
-<param name="mdPadPad" value="8mil"/>
-<param name="mdPadVia" value="8mil"/>
-<param name="mdViaVia" value="8mil"/>
-<param name="mdSmdPad" value="8mil"/>
-<param name="mdSmdVia" value="8mil"/>
-<param name="mdSmdSmd" value="8mil"/>
+<param name="mtCopper" value="0.0356mm 0.0356mm 0.0356mm 0.0356mm 0.0356mm 0.0356mm 0.0356mm 0.0356mm 0.0356mm 0.0356mm 0.0356mm 0.0356mm 0.0356mm 0.0356mm 0.0356mm 0.0356mm"/>
+<param name="mtIsolate" value="1.5011mm 0.1499mm 0.2007mm 0.1499mm 0.2007mm 0.1499mm 0.2007mm 0.1499mm 0.2007mm 0.1499mm 0.2007mm 0.1499mm 0.2007mm 0.1499mm 0.2007mm"/>
+<param name="mdWireWire" value="6mil"/>
+<param name="mdWirePad" value="6mil"/>
+<param name="mdWireVia" value="6mil"/>
+<param name="mdPadPad" value="6mil"/>
+<param name="mdPadVia" value="6mil"/>
+<param name="mdViaVia" value="6mil"/>
+<param name="mdSmdPad" value="6mil"/>
+<param name="mdSmdVia" value="6mil"/>
+<param name="mdSmdSmd" value="6mil"/>
 <param name="mdViaViaSameLayer" value="8mil"/>
 <param name="mnLayersViaInSmd" value="2"/>
-<param name="mdCopperDimension" value="40mil"/>
-<param name="mdDrill" value="8mil"/>
+<param name="mdCopperDimension" value="15mil"/>
+<param name="mdDrill" value="6mil"/>
 <param name="mdSmdStop" value="0mil"/>
-<param name="msWidth" value="10mil"/>
-<param name="msDrill" value="24mil"/>
-<param name="msMicroVia" value="9.99mm"/>
+<param name="msWidth" value="6mil"/>
+<param name="msDrill" value="13mil"/>
+<param name="msMicroVia" value="13mil"/>
 <param name="msBlindViaRatio" value="0.5"/>
 <param name="rvPadTop" value="0.25"/>
@@
 <param name="rvMicroViaOuter" value="0.25"/>
 <param name="rvMicroViaInner" value="0.25"/>
-<param name="rlMinPadTop" value="10mil"/>
+<param name="rlMinPadTop" value="7mil"/>
 <param name="rlMaxPadTop" value="20mil"/>
-<param name="rlMinPadInner" value="10mil"/>
+<param name="rlMinPadInner" value="7mil"/>
 <param name="rlMaxPadInner" value="20mil"/>
-<param name="rlMinPadBottom" value="10mil"/>
+<param name="rlMinPadBottom" value="7mil"/>
 <param name="rlMaxPadBottom" value="20mil"/>
-<param name="rlMinViaOuter" value="8mil"/>
+<param name="rlMinViaOuter" value="7mil"/>
 <param name="rlMaxViaOuter" value="20mil"/>
-<param name="rlMinViaInner" value="8mil"/>
+<param name="rlMinViaInner" value="7mil"/>
 <param name="rlMaxViaInner" value="20mil"/>
 <param name="rlMinMicroViaOuter" value="4mil"/>
@@
 <param name="mlMinCreamFrame" value="0mil"/>
 <param name="mlMaxCreamFrame" value="0mil"/>
-<param name="mlViaStopLimit" value="0mil"/>
+<param name="mlViaStopLimit" value="100mil"/>
 <param name="srRoundness" value="0"/>
 <param name="srMinRoundness" value="0mil"/>
@@
 </elements>
 <signals>
+<signal name="S$1">
+<polygon width="0" layer="16" thermals="no">
+<vertex x="0" y="3"/>
+<vertex x="0" y="32" curve="-90"/>
+<vertex x="3" y="35"/>
+<vertex x="36" y="35"/>
+<vertex x="130" y="35" curve="-90"/>
+<vertex x="133" y="32"/>
+<vertex x="133" y="12"/>
+<vertex x="133" y="3" curve="-90"/>
+<vertex x="130" y="0"/>
+<vertex x="68" y="0"/>
+<vertex x="3" y="0" curve="-90"/>
+</polygon>
+</signal>
 </signals>
 </board>
