File: cyclops/pcb/cyclops.sch (EAGLE design)
At the start: 164 parts, among them Q2 IRF510, U1 MCP4921, U10 OPA1664, U11 THS4281, U12 MAX4564, U13 ZXTD, U14 ZXTD, U4 LT1931, U5 LT1764A, U6 337L, U67 ZLDO1117, U74 TLV3701, U75 LT1711, U8 ADR03, U9 OP1177

Commit message: More circuit revisions.
Parts:
- removed +5V, -1.25V, REF2.5, REF5.0: TPTP16R, cyclops:TPTP16R
- removed C40: .1uF, cyclops:C_0603
- removed J_CS0, J_T0: 0, cyclops:R_0603
- removed J_L5, J_L6: MPZ1608, cyclops:L_0603
- removed Q5: (no value), jonnew:N-MOSFET_SOT23-GSD
- removed U$75: (no value), jonnew:SPST_IC_SOT23-6
- removed U67: ZLDO1117, jonnew:LDO-FIXED_SOT223
- removed U75: LT1711, jonnew:LT1711
- added +6V, -2.5V, REF2.1, REF5.1: TPTP16R, cyclops:TPTP16R
- added C39: 10nF, cyclops:C_0603
- added C7: 100uF, cyclops:C-POL_0807
- added J_CS4, J_T4, R49: 0, cyclops:R_0603
- added J_L1, J_L2: MPZ1608, cyclops:L_0603
- added Q4: IRF510, cyclops:N-MOSFETTO-262
- added R39, R50: (no value), cyclops:R_0603
- added R51: 10k, cyclops:R_0603
- added U15: OPA1664, jonnew:QUAD-OPAMP_14PIND
- added U2: LT1931, cyclops:LT1611
- added U3: LT1764A, cyclops:LT1963_DDPAK
- C11: value 1uF -> 22uF; device cyclops:C_1206 -> cyclops:C_1210
- C12: value 220pF -> 10uF; device cyclops:C_0603 -> jonnew:C_1206
- C13: value 100uF -> 10uF; device cyclops:C-POL_0807 -> jonnew:C_1206
- C14: value 0.1uF -> 10uF; device cyclops:C_0603 -> jonnew:C_1206
- C15: value 22uF -> 10nF; device cyclops:C_1210 -> cyclops:C_1206
- C16: value 1uF -> 10uF; device cyclops:C-POL_1206 -> jonnew:C_1206
- C17: value 1uF -> .1uF; device cyclops:C-POL_1206 -> cyclops:C_0603
- C20, C21: value 1uF -> .1uF; device cyclops:C_0805 -> cyclops:C_0603
- C22, C25, C31, C5: value .1uF -> 1uF; device cyclops:C_0603 -> cyclops:C_0805
- C27, C28: value 1uF -> 0.1uF; device cyclops:C_0805 -> cyclops:C_0603
- C29, C35: value 10nF -> .1uF
- C3: value .1uF -> 10uF; device cyclops:C_0603 -> cyclops:C_1206
- C32: value 220pF -> 1uF; device cyclops:C_0603 -> cyclops:C_0805
- C33: value 10uF -> 10nF; device cyclops:C_1206 -> cyclops:C_0603
- C34, C4: value 10uF -> .1uF; device cyclops:C_1206 -> cyclops:C_0603
- C36: value 0.1uF -> 220pF
- C37, C38: value 1uF -> 10uF; device cyclops:C_0805 -> cyclops:C_1206
- C6: value 1uF -> 4.7uF; device cyclops:C_0805 -> cyclops:C_1206
- C8: value .1uF -> 1uF; device cyclops:C_0603 -> cyclops:C_1206
- C9: value 4.7uF -> 220pF; device cyclops:C_1206 -> cyclops:C_0603
- D1: value MM3Z5V1 -> 1N5819; device cyclops:Z-DIODE_SOD-323 -> jonnew:S-DIODESOD-123
- D2: value MBR0520L -> 1N5819; device cyclops:S-DIODESOD-123 -> jonnew:S-DIODESOD-123
- D3: value 1N5819 -> MM3Z5V1; device jonnew:S-DIODESOD-123 -> cyclops:Z-DIODE_SOD-323
- D4: value 1N5819 -> MBR0520L; device jonnew:S-DIODESOD-123 -> cyclops:S-DIODESOD-123
- Q2: value IRF510 -> (none); device cyclops:N-MOSFETTO-262 -> jonnew:N-MOSFET_SOT23-GSD
- R1: value 10k -> 110k
- R10: value 3k -> 100
- R11: value 10k -> 29.4k
- R12, R3: value 110k -> 10k
- R15: value 1k -> 3k
- R16, R20: value 1k -> 10k
- R17: value 1k -> 40k
- R18, R24: value 1k -> 100k
- R19: value 470 -> 100
- R21: value 110k -> 100k
- R22: value 0 -> 1k
- R23, R28, R32: value 2.2k -> 1k
- R25: value 220k -> 100k
- R26, R30: value (none) -> 1k
- R27: value 220k -> 1k
- R29: value 0 -> 100k
- R31: value 2.2k -> 470
- R33, R34: value 0.5 -> 1k
- R35: value 10k -> 220k
- R36, R43: value 1k -> 0
- R38, R46: value 100k -> 2.2k
- R4: value (none) -> 50; device cyclops:R_0603 -> jonnew:R_1206
- R40: value 100k -> 1k
- R41: value 0 -> 220k
- R42: value 1k -> 2.2k
- R44: value 100 -> (none)
- R45: value (none) -> 2.2k
- R47, R48: value 100k -> 0.5
- R5: value 100 -> 50; device cyclops:R_0603 -> jonnew:R_1206
- R6: value 29.4k -> 50; device cyclops:R_0603 -> jonnew:R_1206
- R7: value 10k -> 50; device cyclops:R_0603 -> jonnew:R_1206
- R8: value 2.15k -> 110k
- R9: value 240 -> (none)
- U10: value OPA1664 -> (none); device cyclops:QUAD-OPAMP_14PIND -> jonnew:SPST_IC_SOT23-6
- U11: device cyclops:OPAMP_SOT-23 -> jonnew:OPAMP_SOT-23
- U4: value LT1931 -> BD60HC5WEFJ; device cyclops:LT1611 -> jonnew:LDO_ADJUST_BDXXHC5WEFJ
- U5: value LT1764A -> TPS72325; device cyclops:LT1963_DDPAK -> jonnew:LDO_ADJUST_TPS72325
- U6: value 337L -> LT1711; device cyclops:337L -> jonnew:LT1711
- U9: value OP1177 -> LT1880; device cyclops:OP1177ARMZ -> jonnew:OPAMP_SOT-23
- renumbered J_ADDR0 to J_ADDR4, J_LDAC0 to J_LDAC4, J_OC0 to J_OC4, L7 to L3, L8 to L4, U74 to U7
Connections:
- removed net +12V: AUX<FB>CURR.3, C13.+, C19.1, C20.1, C21.1, C22.1, C23.1, C25.1, C27.1, C30.1, C34.1, C38.1, EXPANSION.7, Q2.D, R10.2, R12.1, R15.2, R16.2, R25.2, R31.1, R42.2, R8.2, U10P.V+, U11G$2.V+, U13G$1.C, U14G$1.C, U5.VO, U67.VI, U7G$2.V+, U8.VIN, U9.V+
- removed net +5V: +5V.TP, C35.1, C36.1, C37.1, C5.1, C6.1, C8.1, L2.2, U$75.V+, U1.VDD, U12.V+, U67.VO, U75G$2.V+
- removed net -1.25V: -1.25V.TP, C14.1, C17.-, C26.1, C28.1, C29.1, C3.1, C31.1, C33.1, R27.1, R32.2, U$75.V-, U10P.V-, U11G$2.V-, U12.V-, U13G$2.C, U14G$2.C, U6.VO, U75G$2.V-
- new net +13.3V: C10.+, C12.1, C34.1, C38.1, EXPANSION.7, Q4.D, R13.2, R15.2, R45.1, U11G$2.V+, U13G$1.C, U14G$1.C, U3.VO, U4.EN, U4.VI
- new net +6V: +6V.TP, AUX<FB>CURR.3, C14.1, C19.1, C20.1, C22.1, C23.1, C28.1, C29.1, C31.1, C39.1, C4.1, C5.1, L1.2, R26.2, R27.2, R30.2, R35.2, U1.VDD, U10.V+, U12.V+, U15P.V+, U6G$2.V+, U7G$2.V+, U8.VIN
- new net -2.5V: -2.5V.TP, C15.2, C16.2, C21.1, C27.1, C30.1, C32.1, C33.1, C35.1, C37.1, R41.1, R46.2, U10.V-, U11G$2.V-, U12.V-, U13G$2.C, U14G$2.C, U15P.V-, U5.VO, U6G$2.V-
- new net N$48: C13.1, C16.1, U5.GND
- new net N$51: C15.1, U5.ADJ/NR
- new net N$52: R4.1, VAUX_OUT.1
- new net N$53: R5.1, VAUX_IN.1
- new net N$54: R6.1, VI.1
- new net N$55: R7.1, VREF.1
- new net N$57: C24.2
- new net V+: C24.1, C25.1, U9G$2.V+
- net +15V: now also C7.+, U3.VI, U3.~SHDN; no longer C10.+, U5.VI, U5.~SHDN
- net +3V3: now also R3.1; no longer R1.1
- net -5V: now also C13.2, U5.EN, U5.VI; no longer C16.-, U6.VI
- net COM: now also C36.1; no longer C32.1
- net COMP+: now also C17.1, R16.1; no longer C18.1, R11.1
- net CS: now also J_CS2.1, J_CS4.2; no longer J_CS0.1, J_CS2.2
- net CS0: now also J_CS2.2; no longer J_CS0.2
- net CS2: now also J_CS3.1; no longer J_CS2.1
- net CS3: now also J_CS4.1; no longer J_CS3.1
- net DACA: now also R9.2; no longer R4.2
- net GND: now also C11.2, C12.2, C17.2, C32.2, C39.2, C7.-, D3.A, D4.C, Q2.S, R12.1, R14.1, R19.1, R24.1, R25.1, R29.1, R32.1, R33.2, R39.2, R42.2, R44.2, R50.2, R51.1, R8.2, U10.GND, U2.GND, U3.GND, U6G$1.GND, U6G$1.LATCH; no longer C13.-, C15.2, C16.+, C17.+, C24.2, C36.2, C40.2, C8.2, C9.2, D1.A, D2.C, Q5.S, R17.2, R20.1, R21.2, R26.2, R28.2, R30.2, R35.1, R44.1, R45.2, R46.1, R47.1, R48.1, R7.1, R9.1, U$75.GND, U4.GND, U5.GND, U6.ADJ, U67.GND, U75G$1.GND, U75G$1.LATCH, U9.V-
- net LDAC1: now also J_LDAC3.2; no longer J_LDAC1.2
- net LDAC3: now also J_LDAC1.2; no longer J_LDAC3.2
- net LED+: now also Q4.S; no longer Q2.S
- net LED-: now also U15A.+IN, U15C.+IN; no longer U10A.+IN, U10C.+IN
- net LED_ACTIVE: now also R23.2, U6G$1.~Q; no longer R43.2, U75G$1.~Q
- net N$1: now also R9.1; no longer R4.1
- net N$10: now also R46.1; no longer R32.1
- net N$11: now also R49.1, R50.1, U15A.-IN; no longer R41.1, R45.1, U10A.-IN
- net N$12: now also R13.1, R14.2, U3.ADJ; no longer R8.1, R9.2, U5.ADJ
- net N$13: now also C36.2, R42.1; no longer C32.2, R28.1
- net N$14: now also R10.1; no longer R5.1
- net N$15: now also R43.1, R44.1, U15C.-IN; no longer R29.1, R30.1, U10C.-IN
- net N$16: now also R30.1; no longer R16.1
- net N$18: now also R33.1, R34.2, U9G$1.-IN; no longer R17.1, R18.2, U9.-IN
- net N$19: now also J_L3.1; no longer J_L5.1
- net N$2: now also R26.1; no longer R15.1
- net N$20: now also R31.2; no longer R19.2
- net N$21: now also J_L2.1; no longer J_L4.1
- net N$22: now also R31.1; no longer R19.1
- net N$23: now also J_L1.1; no longer J_L3.1
- net N$24: now also R48.1; no longer R34.1
- net N$25: now also R47.1; no longer R33.1
- net N$26: now also Q4.G, R47.2, R48.2, R51.2; no longer Q2.G, R33.2, R34.2, R35.2
- net N$27: now also R22.2; no longer R14.2
- net N$28: now also R22.1, R24.2; no longer R14.1, R47.2
- net N$3: now also R15.1; no longer R10.1
- net N$32: now also C8.1, U2.SW; no longer C11.1, U4.SW
- net N$33: now also C8.2, D4.A; no longer C11.2, D2.A
- net N$35: now also C11.1, C9.1, R11.2; no longer C12.1, C15.1, R6.2
- net N$36: now also C9.2, R11.1, R12.2, U2.NFB; no longer C12.2, R6.1, R7.2, U4.NFB
- net N$37: now also R40.1; no longer R24.1
- net N$38: now also L2.2, R8.1; no longer L1.2, R21.1
- net N$39: now also R28.1, R29.2; no longer R36.1, R48.2
- net N$4: now also R45.2; no longer R31.2
- net N$40: now also J_ADDR1.2; no longer J_ADDR3.2
- net N$42: now also R18.1, R19.2, R21.1, U6G$1.+IN; no longer R38.1, R40.1, R44.2, U75G$1.+IN
- net N$43: now also D2.A, L1.1; no longer D3.A, L2.1
- net N$44: now also J_ADDR3.2; no longer J_ADDR1.2
- net N$46: now also R27.1; no longer R42.1
- net N$47: now also Q2.D; no longer Q5.D
- net N$49: now also Q2.G, R23.1, R25.2; no longer Q5.G, R43.1, R46.2
- net N$5: now also C18.1, R17.2, R20.1; no longer C40.1, R12.2, R13.1
- net N$50: now also R21.2, U6G$1.Q; no longer R38.2, U75G$1.Q
- net N$6: now also R32.2; no longer R20.2
- net N$7: now also J_L4.1; no longer J_L6.1
- net N$8: now also R36.1, R39.1, U15D.-IN; no longer R22.1, R26.1, U10D.-IN
- net OC1: now also J_OC3.2; no longer J_OC1.2
- net OC3: now also J_OC1.2; no longer J_OC3.2
- net OVER_CURR: now also L2.1, R28.2; no longer L1.1, R36.2
- net REF2.5: now also C3.1, REF2.1.TP, U9G$1.+IN; no longer C4.1, REF2.5.TP, U9.+IN
- net REF5.0: now also C26.1, R17.1, R18.2, R34.1, REF5.1.TP, U9G$1.OUT; no longer C24.1, R18.1, R40.2, REF5.0.TP, U9.OUT
- net SCL: now also R2.2; no longer R1.2
- net SDA: now also R3.2; no longer R2.2
- net T0: now also J_T1.1; no longer J_T0.1
- net T1: now also J_T2.1; no longer J_T1.1
- net T2: now also J_T3.1; no longer J_T2.1
- net T3: now also J_T4.1; no longer J_T3.1
- net TRIG: now also J_T4.2; no longer J_T0.2
- net V-: now also R20.2, U9G$2.V-; no longer R13.2
- net VAUX: now also R35.1, R5.2, U15B.+IN; no longer R25.1, U10B.+IN, VAUX_IN.1
- net VAUX_OUT: now also R4.2, U15B.-IN, U15B.OUT; no longer U10B.-IN, U10B.OUT, VAUX_OUT.1
- net VCTL: now also D3.C, R10.2, U10.S; no longer D1.C, R5.2, U$75.S
- net VCTL_PROT: now also R38.2, U10.D; no longer R23.2, U$75.D
- net VCTL_PROTECT: now also R38.1; no longer R23.1
- net VI: now also R43.2, R6.2, U15C.OUT; no longer R29.2, U10C.OUT, VI.1
- net VIN: now also C6.1, D2.C, U2.VIN, U2.~SHDN; no longer C9.1, D3.C, U4.VIN, U4.~SHDN
- net VI_INTERNAL: now also R1.1, R16.2, R49.2, U15A.OUT, U6G$1.-IN; no longer R11.2, R3.1, R41.2, U10A.OUT, U75G$1.-IN
- net VI_LP: now also J_L1.2, J_L2.2, R1.2; no longer J_L5.2, J_L6.2, R3.2
- net VREF: now also R36.2, U15D.OUT; no longer R22.2, U10D.OUT
- net VREF/TTL: now also R7.2; no longer VREF.1
- net _VREF: now also R40.2, R41.2, U15D.+IN; no longer R24.2, R27.2, U10D.+IN
Other:
- note added: "LED ACTIVE (I_LED >10 mA)"
- note removed: "LED ACTIVE (>10 mA)"
- note removed: "OR +12V.."
