File: cyclops/pcb/cyclops.sch (EAGLE design)
At the start: 178 parts, among them Q4 IRF510, U1 MCP4921, U11 THS4281, U12 MAX4564, U13 ZXTD, U14 ZXTD, U15 OPA1664, U2 LT1931, U3 LT1764A, U31 TPS62153, U4 BD00IA5WEFJ-E2, U5 TPS72325, U6 LT1711, U7 TLV3701, U8 ADR03, U9 LT1880

Commit message: Started ERC/DRC process.
Parts:
- added +13.3V, GND: RCU-0C, jonnew:TP_RC0603
- +5V, +6V, -2.5V, -5V, REF2V5, REF5V0: value TPTP16R -> RCU-0C; device cyclops:TPTP16R -> jonnew:TP_RC0603
- IND, OC: value (none) -> 569-0112-200
- Q1, Q2, Q3: value (none) -> SSM3K324
- U10: value (none) -> ADG1201
Connections:
- net +13.3V: now also +13.3V.TP
- net GND: now also GND.TP, UC.AGND
Changed lines of the file:
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@@
 <part name="Q4" library="cyclops" deviceset="N-MOSFET" device="TO-262" value="IRF510"/>
 <part name="VAUX_OUT" library="jonnew" deviceset="BNC" device="_0731000105" value="0731000105"/>
-<part name="REF2V5" library="cyclops" deviceset="TP" device="TP16R" value="TPTP16R"/>
-<part name="REF5V0" library="cyclops" deviceset="TP" device="TP16R" value="TPTP16R"/>
+<part name="REF2V5" library="jonnew" deviceset="TP" device="_RC0603" value="RCU-0C"/>
+<part name="REF5V0" library="jonnew" deviceset="TP" device="_RC0603" value="RCU-0C"/>
 <part name="R15" library="cyclops" deviceset="R" device="_0603" value="2.2k"/>
 <part name="R20" library="cyclops" deviceset="R" device="_0603" value="10k"/>
@@
 <part name="P-6" library="cyclops" deviceset="-5V" device="" value="-2.5V"/>
 <part name="C36" library="cyclops" deviceset="C" device="_0603" value="220pF"/>
-<part name="-5V" library="cyclops" deviceset="TP" device="TP16R" value="TPTP16R"/>
-<part name="-2.5V" library="cyclops" deviceset="TP" device="TP16R" value="TPTP16R"/>
+<part name="-5V" library="jonnew" deviceset="TP" device="_RC0603" value="RCU-0C"/>
+<part name="-2.5V" library="jonnew" deviceset="TP" device="_RC0603" value="RCU-0C"/>
 <part name="VPRE" library="cyclops" deviceset="TP" device="TP16R" value="TPTP16R"/>
 <part name="C27" library="cyclops" deviceset="C" device="_0603" value="0.1uF"/>
@@
 <part name="J_OC0" library="jonnew" deviceset="R" device="_0402" value="0"/>
 <part name="R37" library="cyclops" deviceset="R" device="_0603" value="0"/>
-<part name="IND" library="jonnew" deviceset="LED_2X" device="_VERTICAL"/>
-<part name="OC" library="jonnew" deviceset="LED_2X" device="_VERTICAL"/>
+<part name="IND" library="jonnew" deviceset="LED_2X" device="_VERTICAL" value="569-0112-200"/>
+<part name="OC" library="jonnew" deviceset="LED_2X" device="_VERTICAL" value="569-0112-200"/>
 <part name="D2" library="jonnew" deviceset="S-DIODE" device="SOD-123" value="1N5819"/>
 <part name="VREF&lt;&gt;TTL" library="jonnew" deviceset="SPDT" device="_AS12A*" value="JS102"/>
@@
 <part name="C12" library="jonnew" deviceset="C" device="_1206" value="10uF"/>
 <part name="P+4" library="jonnew" deviceset="+5V" device="" value="+6V"/>
-<part name="+6V" library="cyclops" deviceset="TP" device="TP16R" value="TPTP16R"/>
+<part name="+6V" library="jonnew" deviceset="TP" device="_RC0603" value="RCU-0C"/>
 <part name="C18" library="cyclops" deviceset="C" device="_0603" value=".1uF"/>
 <part name="U$64" library="cyclops" deviceset="GND2" device=""/>
@@
 <part name="J_ADDR2" library="jonnew" deviceset="R" device="_0402" value="0"/>
 <part name="J_ADDR3" library="jonnew" deviceset="R" device="_0402" value="0"/>
-<part name="Q1" library="jonnew" deviceset="N-MOSFET" device="_SOT23-GSD"/>
-<part name="Q3" library="jonnew" deviceset="N-MOSFET" device="_SOT23-GSD"/>
-<part name="Q2" library="jonnew" deviceset="N-MOSFET" device="_SOT23-GSD"/>
+<part name="Q1" library="jonnew" deviceset="N-MOSFET" device="_SOT23-GSD" value="SSM3K324"/>
+<part name="Q3" library="jonnew" deviceset="N-MOSFET" device="_SOT23-GSD" value="SSM3K324"/>
+<part name="Q2" library="jonnew" deviceset="N-MOSFET" device="_SOT23-GSD" value="SSM3K324"/>
 <part name="P-8" library="cyclops" deviceset="-5V" device="" value="-2.5V"/>
 <part name="C21" library="cyclops" deviceset="C" device="_0603" value=".1uF"/>
@@
 <part name="P+1" library="jonnew" deviceset="+5V" device="" value="+6V"/>
 <part name="P+5" library="jonnew" deviceset="+5V" device="" value="+6V"/>
-<part name="U10" library="jonnew" deviceset="SPST_IC" device="_SOT23-6"/>
+<part name="U10" library="jonnew" deviceset="SPST_IC" device="_SOT23-6" value="ADG1201"/>
 <part name="P+9" library="jonnew" deviceset="+5V" device="" value="+6V"/>
 <part name="P+10" library="jonnew" deviceset="+5V" device="" value="+6V"/>
@@
 <part name="U$74" library="cyclops" deviceset="GND1" device=""/>
 <part name="U$75" library="cyclops" deviceset="GND1" device=""/>
-<part name="+5V" library="cyclops" deviceset="TP" device="TP16R" value="TPTP16R"/>
+<part name="+5V" library="jonnew" deviceset="TP" device="_RC0603" value="RCU-0C"/>
 <part name="U$76" library="cyclops" deviceset="GND1" device=""/>
 <part name="R5" library="cyclops" deviceset="R" device="_0603" value="33k"/>
@@
 <part name="P+19" library="cyclops" deviceset="+5V" device="" value="+6V"/>
 <part name="L1" library="cyclops" deviceset="L" device="_0603" value="MPZ1608"/>
+<part name="GND" library="jonnew" deviceset="TP" device="_RC0603" value="RCU-0C"/>
+<part name="U$79" library="cyclops" deviceset="GND2" device=""/>
+<part name="+13.3V" library="jonnew" deviceset="TP" device="_RC0603" value="RCU-0C"/>
 </parts>
 <sheets>
@@
 <wire x1="-12.7" y1="149.86" x2="-12.7" y2="190.5" width="0.4064" layer="97" style="shortdash"/>
 <text x="-7.62" y="185.42" size="3.81" layer="97">Teensy components</text>
+<text x="208.28" y="40.64" size="1.6764" layer="97" rot="R90">DNP</text>
+<text x="208.28" y="30.48" size="1.6764" layer="97" rot="R90">DNP</text>
 </plain>
 <instances>
@@
 <attribute name="VALUE" x="12.7" y="87.63" size="1.778" layer="96"/>
 </instance>
+<instance part="GND" gate="G$1" x="68.58" y="-22.86"/>
+<instance part="U$79" gate="G$1" x="68.58" y="-33.02"/>
 </instances>
 <busses>
@@
 <segment>
 <wire x1="127" y1="121.92" x2="127" y2="114.3" width="0.1524" layer="91"/>
-<wire x1="116.84" y1="121.92" x2="127" y2="121.92" width="0.1524" layer="91"/>
+<wire x1="116.84" y1="121.92" x2="121.92" y2="121.92" width="0.1524" layer="91"/>
 <pinref part="UC" gate="G$1" pin="GND"/>
+<pinref part="UC" gate="G$1" pin="AGND"/>
+<wire x1="121.92" y1="121.92" x2="127" y2="121.92" width="0.1524" layer="91"/>
+<wire x1="116.84" y1="109.22" x2="121.92" y2="109.22" width="0.1524" layer="91"/>
+<wire x1="121.92" y1="109.22" x2="121.92" y2="121.92" width="0.1524" layer="91"/>
+<junction x="121.92" y="121.92"/>
 </segment>
 <segment>
@@
 <pinref part="D6" gate="G$1" pin="A"/>
 <wire x1="20.32" y1="-63.5" x2="20.32" y2="-60.96" width="0.1524" layer="91"/>
+</segment>
+<segment>
+<pinref part="GND" gate="G$1" pin="TP"/>
+<wire x1="68.58" y1="-25.4" x2="68.58" y2="-30.48" width="0.1524" layer="91"/>
 </segment>
 </net>
@@
 <instance part="R5" gate="R" x="114.3" y="27.94" rot="R90"/>
 <instance part="R52" gate="R" x="114.3" y="10.16" rot="R90"/>
+<instance part="+13.3V" gate="G$1" x="7.62" y="43.18"/>
 </instances>
 <busses>
@@
 <junction x="58.42" y="38.1"/>
 <wire x1="27.94" y1="38.1" x2="58.42" y2="38.1" width="0.1524" layer="91"/>
+<pinref part="+13.3V" gate="G$1" pin="TP"/>
+<wire x1="7.62" y1="40.64" x2="7.62" y2="38.1" width="0.1524" layer="91"/>
+<junction x="71.12" y="38.1"/>
 </segment>
 </net>
@@
 <junction x="-38.1" y="-17.78"/>
 <pinref part="REF2V5" gate="G$1" pin="TP"/>
+<label x="-27.94" y="-17.78" size="1.778" layer="95"/>
 </segment>
 </net>
@@
 <junction x="139.7" y="20.32"/>
 <pinref part="U15" gate="A" pin="+IN"/>
+<label x="165.1" y="40.64" size="1.778" layer="95"/>
 </segment>
 </net>
@@
 <wire x1="165.1" y1="96.52" x2="165.1" y2="86.36" width="0.1524" layer="91"/>
 <pinref part="LED+" gate="G$1" pin="1"/>
-</segment>
-</net>
+<label x="165.1" y="88.9" size="1.778" layer="95"/>
+</segment>
+</net>
