File: cyclops/pcb/cyclops.sch (EAGLE design)
At the start: 180 parts, among them Q1 SSM3K324, Q2 SSM3K324, Q3 SSM3K324, Q4 IRF510, U1 MCP4921, U10 ADG1201, U11 THS4281, U12 MAX4564, U13 ZXTD, U14 ZXTD, U15 OPA1664, U2 LT1931, U3 LT1764A, U31 TPS62153, U4 BD00IA5WEFJ, U5 TPS72325, U6 LT1711, U7 TLV3701, U8 ADR03, U9 LT1880

Commit message: Rev 3.6 alpha ready for fabrication.
Connections:
- net CS2: now also UC.20/A6/PWM; no longer UC.21/A7/PWM
- net CS3: now also UC.21/A7/PWM; no longer UC.20/A6/PWM
Other:
- note removed: "TODO: 1. ~~Replace arduino headers with teensy headers (male and female since teensy comes without them)~~ 2. ~~Are the LED arrays mounted at correct distance from board edge?~~ 3.~~ Is teensy at correct distance from board edge?~~ 4. ~~Is there adequare clearance b/w rear panel mount components~~ 5. Rearrange panels to fit changes in front and back 6. ~~+5V regulator layou EDIT: +6V~~ 7. ~~Test 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"
- moved on the sheet: J_CS2, J_CS3
Changed lines of the file:
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@@
 <attribute name="DESIGNER" value="JONATHAN P. NEWMAN"/>
 <attribute name="DOC_NUMBER" value="N/A"/>
-<attribute name="REVISION" value="3.5D"/>
+<attribute name="REVISION" value="3.6"/>
 </attributes>
 <variantdefs>
@@
 <part name="U$62" library="cyclops" deviceset="GND1" device=""/>
 <part name="R28" library="cyclops" deviceset="R" device="_0603" value="1k"/>
+<part name="J_CS3" library="jonnew" deviceset="R" device="_0402" value="0"/>
 <part name="J_CS2" library="jonnew" deviceset="R" device="_0402" value="0"/>
-<part name="J_CS3" library="jonnew" deviceset="R" device="_0402" value="0"/>
 <part name="J_CS1" library="jonnew" deviceset="R" device="_0402" value="0"/>
 <part name="J_CS0" library="jonnew" deviceset="R" device="_0402" value="0"/>
@@
 <part name="U$28" library="cyclops" deviceset="GND2" device=""/>
 <part name="U$48" library="jonnew" deviceset="TEENSY-2X7-PIN-HEADER" device="" value="SSQ-107-03-G-D"/>
-<part name="U$54" library="jonnew" deviceset="TEENSY-3-PIN-HEADER" device="" value="SSQ-103-03-G-S"/>
+<part name="U$54" library="jonnew" deviceset="TEENSY-2-PIN-HEADER" device="" value="SSQ-102-03-G-S"/>
 <part name="U$55" library="jonnew" deviceset="TEENSY-14-PIN-HEADER" device="" value="SSQ-114-03-G-S"/>
 <part name="U$63" library="jonnew" deviceset="TEENSY-14-PIN-HEADER" device="" value="SSQ-114-03-G-S"/>
 <part name="D1" library="jonnew" deviceset="S-DIODE" device="SOD-123" value="1N5819"/>
 <part name="U$66" library="jonnew" deviceset="TEENSY-2X7-PIN-HEADER" device="" value="NPTC072KFMS-RC"/>
-<part name="U$69" library="jonnew" deviceset="TEENSY-3-PIN-HEADER" device="" value="PPPC031LFBN-RC"/>
 <part name="U$72" library="jonnew" deviceset="TEENSY-14-PIN-HEADER" device="" value="PPPC141LFBN-RC"/>
 <part name="U$73" library="jonnew" deviceset="TEENSY-14-PIN-HEADER" device="" value="PPPC141LFBN-RC"/>
@@
 <part name="+13.3V" library="jonnew" deviceset="TP" device="_RC0603" value="RCU-0C"/>
 <part name="C40" library="cyclops" deviceset="C" device="_1210" value="22uF"/>
+<part name="U$80" library="jonnew" deviceset="TEENSY-2-PIN-HEADER" device="" value="PPPC021LFBN-RC"/>
 </parts>
 <sheets>
@@
 <wire x1="17.78" y1="17.78" x2="17.78" y2="99.06" width="0.4064" layer="97" style="shortdash"/>
 <wire x1="17.78" y1="99.06" x2="-7.62" y2="99.06" width="0.4064" layer="97" style="shortdash"/>
-<text x="76.2" y="149.86" size="2.54" layer="97">TODO:
-1. ~~Replace arduino headers with teensy headers (male and female since teensy comes without them)~~
-2. ~~Are the LED arrays mounted at correct distance from board edge?~~
-3.~~ Is teensy at correct distance from board edge?~~
-4. ~~Is there adequare clearance b/w rear panel mount components~~
-5. Rearrange panels to fit changes in front and back
-6. ~~+5V regulator layou EDIT: +6V~~
-7. ~~Test LED ON circuit. You will at least have to replace the N BJT with an P BJT since LED ON is inverted.~~
-8. ~~Teensy itself will need to be modified with cut trace and schottky diode to work with external power~~
-9. ~~Replace SMD VREF/TTL switch with vertical slide like 360‑3344‑ND~~
-10. ~~Bring +12V up to +13.5 and -1.5 to -2.5V if possible. Examine components to see what is limiting the positive/negative rails.~~
-11. ~~Stripline calculations and proper terminations for new high-side analog drive train and new analog switch (thinking about replacing drive train MAX4564 with ADV3220 which provides 800 MHz -3dB and 2x gain hardcoded). EDIT: 11 mil is good when using top layer and 2nd layer ground for circuit hub PCBs~~
-12. ~~Rename jumper resistors~~
-13. ~~Replace +6V LDO with something that can actually handle +13.3V input. Place close to 13.3V LDO. Add buck converter to digital power supply to provide fixed 5V for teensy and to power inverter. 15V should be routed to digital section on bottom layer of board along the bottom edge of board. Ground should be cut along the top edge of this trace to force digital power return back to 15V jack along this trace, away from analog stuff.~~
-14. ~~Protect inputs of opa1664 with schottkys~~
-15. ~~TTL/VREF switch pin overlaps with heatsink.~~
-16. Remove unused vref pin from teensy so that thta TRIG BNC has plenty of room. Update the headers to be 2 pin instead of 3</text>
 <wire x1="-12.7" y1="190.5" x2="71.12" y2="190.5" width="0.4064" layer="97" style="shortdash"/>
 <wire x1="71.12" y1="190.5" x2="71.12" y2="149.86" width="0.4064" layer="97" style="shortdash"/>
@@
 </instance>
 <instance part="U$62" gate="G$1" x="160.02" y="76.2"/>
-<instance part="J_CS2" gate="R" x="43.18" y="76.2" smashed="yes" rot="R180">
+<instance part="J_CS3" gate="R" x="43.18" y="76.2" smashed="yes" rot="R180">
 <attribute name="NAME" x="46.99" y="76.4286" size="1.778" layer="95"/>
 </instance>
-<instance part="J_CS3" gate="R" x="43.18" y="78.74" smashed="yes" rot="R180">
+<instance part="J_CS2" gate="R" x="43.18" y="78.74" smashed="yes" rot="R180">
 <attribute name="NAME" x="46.99" y="78.9686" size="1.778" layer="95"/>
 </instance>
@@
 <instance part="D1" gate="G$1" x="7.62" y="160.02" rot="R180"/>
 <instance part="U$66" gate="G$1" x="50.8" y="177.8" rot="R270"/>
-<instance part="U$69" gate="G$1" x="50.8" y="165.1" rot="R270"/>
 <instance part="U$72" gate="G$1" x="33.02" y="177.8" rot="R270"/>
 <instance part="U$73" gate="G$1" x="33.02" y="165.1" rot="R270"/>
@@
 <instance part="GND" gate="G$1" x="68.58" y="-22.86"/>
 <instance part="U$79" gate="G$1" x="68.58" y="-33.02"/>
+<instance part="U$80" gate="G$1" x="50.8" y="165.1" rot="R270"/>
 </instances>
 <busses>
@@
 <wire x1="38.1" y1="106.68" x2="33.02" y2="106.68" width="0.1524" layer="91"/>
 <wire x1="33.02" y1="104.14" x2="33.02" y2="106.68" width="0.1524" layer="91"/>
-<pinref part="J_CS3" gate="R" pin="2"/>
+<pinref part="J_CS2" gate="R" pin="2"/>
 <wire x1="33.02" y1="78.74" x2="38.1" y2="78.74" width="0.1524" layer="91"/>
 <wire x1="33.02" y1="104.14" x2="33.02" y2="78.74" width="0.1524" layer="91"/>
 <junction x="33.02" y="104.14"/>
 <junction x="33.02" y="78.74"/>
-<pinref part="J_CS2" gate="R" pin="2"/>
+<pinref part="J_CS3" gate="R" pin="2"/>
 <wire x1="33.02" y1="76.2" x2="38.1" y2="76.2" width="0.1524" layer="91"/>
 <wire x1="33.02" y1="78.74" x2="33.02" y2="76.2" width="0.1524" layer="91"/>
@@
 <segment>
 <pinref part="J_CS3" gate="R" pin="1"/>
-<wire x1="48.26" y1="78.74" x2="71.12" y2="78.74" width="0.1524" layer="91"/>
-<label x="60.96" y="78.74" size="1.778" layer="95"/>
-<pinref part="UC" gate="G$1" pin="20/A6/PWM"/>
+<wire x1="48.26" y1="76.2" x2="71.12" y2="76.2" width="0.1524" layer="91"/>
+<label x="60.96" y="76.2" size="1.778" layer="95"/>
+<pinref part="UC" gate="G$1" pin="21/A7/PWM"/>
 </segment>
 </net>
@@
 <segment>
 <pinref part="J_CS2" gate="R" pin="1"/>
-<wire x1="48.26" y1="76.2" x2="71.12" y2="76.2" width="0.1524" layer="91"/>
-<label x="60.96" y="76.2" size="1.778" layer="95"/>
-<pinref part="UC" gate="G$1" pin="21/A7/PWM"/>
-</segment>
-</net>
+<wire x1="48.26" y1="78.74" x2="71.12" y2="78.74" width="0.1524" layer="91"/>
+<label x="60.96" y="78.74" size="1.778" layer="95"/>
+<pinref part="UC" gate="G$1" pin="20/A6/PWM"/>
+</segment>
+</net>
