File: cyclops/pcb/cyclops.brd (EAGLE design)
At the start: 124.5 x 79.9 mm, 183 parts, among them Q1 SSM3K324, Q2 SSM3K324, Q3 SSM3K324, Q4 IRF510, U1 MCP4921, U10 ADG1201, U11 THS4281, U12 MAX4564, U13 ZXTD, U14 ZXTD, U15 OPA1664, U2 LT1931, U3 LT1764A, U31 TPS62153, U4 BD00IA5WEFJ, U5 TPS72325, U6 LT1711, U7 TLV3701, U8 ADR03, U9 LT1880

Commit message: Rev 3.6 alpha ready for fabrication.
Parts:
- moved J_CS3 0.13 mm to (8.38, 39.4)
Connections:
- net CS2: now also UC.20/A6; no longer UC.21/A7
- net CS3: now also UC.21/A7; no longer UC.20/A6
Routing:
- net CS2: track 43.2 -> 47.4 mm, vias 0 -> 2
- net CS3: track 45.4 -> 41.6 mm
Changed lines of the file:
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@@
 <layer number="17" name="Pads" color="2" fill="1" visible="yes" active="yes"/>
 <layer number="18" name="Vias" color="2" fill="1" visible="yes" active="yes"/>
-<layer number="19" name="Unrouted" color="6" fill="1" visible="no" active="yes"/>
+<layer number="19" name="Unrouted" color="6" fill="1" visible="yes" active="yes"/>
 <layer number="20" name="Dimension" color="15" fill="1" visible="yes" active="yes"/>
 <layer number="21" name="tPlace" color="7" fill="1" visible="yes" active="yes"/>
-<layer number="22" name="bPlace" color="7" fill="1" visible="no" active="yes"/>
+<layer number="22" name="bPlace" color="7" fill="1" visible="yes" active="yes"/>
 <layer number="23" name="tOrigins" color="15" fill="1" visible="yes" active="yes"/>
-<layer number="24" name="bOrigins" color="15" fill="1" visible="no" active="yes"/>
+<layer number="24" name="bOrigins" color="15" fill="1" visible="yes" active="yes"/>
 <layer number="25" name="tNames" color="7" fill="1" visible="yes" active="yes"/>
-<layer number="26" name="bNames" color="7" fill="1" visible="no" active="yes"/>
+<layer number="26" name="bNames" color="7" fill="1" visible="yes" active="yes"/>
 <layer number="27" name="tValues" color="7" fill="1" visible="yes" active="yes"/>
-<layer number="28" name="bValues" color="7" fill="1" visible="no" active="yes"/>
-<layer number="29" name="tStop" color="7" fill="3" visible="no" active="yes"/>
-<layer number="30" name="bStop" color="7" fill="6" visible="no" active="yes"/>
+<layer number="28" name="bValues" color="7" fill="1" visible="yes" active="yes"/>
+<layer number="29" name="tStop" color="7" fill="3" visible="yes" active="yes"/>
+<layer number="30" name="bStop" color="7" fill="6" visible="yes" active="yes"/>
 <layer number="31" name="tCream" color="7" fill="4" visible="no" active="yes"/>
 <layer number="32" name="bCream" color="7" fill="5" visible="no" active="yes"/>
@@
 <layer number="37" name="tTest" color="7" fill="1" visible="no" active="yes"/>
 <layer number="38" name="bTest" color="7" fill="1" visible="no" active="yes"/>
-<layer number="39" name="tKeepout" color="4" fill="11" visible="yes" active="yes"/>
-<layer number="40" name="bKeepout" color="1" fill="11" visible="yes" active="yes"/>
-<layer number="41" name="tRestrict" color="4" fill="10" visible="yes" active="yes"/>
-<layer number="42" name="bRestrict" color="1" fill="10" visible="yes" active="yes"/>
-<layer number="43" name="vRestrict" color="2" fill="10" visible="yes" active="yes"/>
-<layer number="44" name="Drills" color="7" fill="1" visible="yes" active="yes"/>
-<layer number="45" name="Holes" color="7" fill="1" visible="yes" active="yes"/>
+<layer number="39" name="tKeepout" color="4" fill="11" visible="no" active="yes"/>
+<layer number="40" name="bKeepout" color="1" fill="11" visible="no" active="yes"/>
+<layer number="41" name="tRestrict" color="4" fill="10" visible="no" active="yes"/>
+<layer number="42" name="bRestrict" color="1" fill="10" visible="no" active="yes"/>
+<layer number="43" name="vRestrict" color="2" fill="10" visible="no" active="yes"/>
+<layer number="44" name="Drills" color="7" fill="1" visible="no" active="yes"/>
+<layer number="45" name="Holes" color="7" fill="1" visible="no" active="yes"/>
 <layer number="46" name="Milling" color="3" fill="1" visible="no" active="yes"/>
 <layer number="47" name="Measures" color="7" fill="1" visible="no" active="yes"/>
@@
 <attribute name="VALUE" x="9.779" y="51.181" size="1.016" layer="27" font="vector" ratio="18" align="center-left"/>
 </element>
+<element name="J_CS3" library="jonnew" package="0402" value="0" x="8.382" y="39.37" smashed="yes"/>
 <element name="J_CS2" library="jonnew" package="0402" value="0" x="8.382" y="40.894" smashed="yes"/>
-<element name="J_CS3" library="jonnew" package="0402" value="0" x="8.382" y="39.243" smashed="yes"/>
 <element name="J_CS1" library="jonnew" package="0402" value="0" x="8.382" y="42.418" smashed="yes" rot="R180"/>
 <element name="J_CS0" library="jonnew" package="0402" value="0" x="8.382" y="43.942" smashed="yes" rot="R180"/>
@@
 <wire x1="24.892" y1="53.467" x2="25.019" y2="53.467" width="0.1778" layer="1"/>
 <contactref element="J_CS1" pad="1"/>
-<contactref element="J_CS3" pad="2"/>
 <contactref element="J_CS2" pad="2"/>
+<contactref element="J_CS3" pad="2"/>
 <wire x1="8.9154" y1="43.942" x2="8.9154" y2="42.418" width="0.127" layer="1"/>
-<wire x1="8.9154" y1="40.894" x2="8.9154" y2="39.243" width="0.127" layer="1"/>
-<wire x1="8.9154" y1="42.418" x2="8.9154" y2="40.894" width="0.127" layer="1"/>
 <wire x1="8.9154" y1="43.942" x2="12.8524" y2="47.879" width="0.127" layer="1"/>
 <wire x1="12.8524" y1="47.879" x2="22.0720125" y2="47.879" width="0.127" layer="1"/>
 <wire x1="22.0720125" y1="47.879" x2="25.019" y2="50.8259875" width="0.127" layer="1"/>
 <wire x1="25.019" y1="50.8259875" x2="25.019" y2="52.518" width="0.127" layer="1"/>
+<wire x1="8.9154" y1="42.418" x2="8.9154" y2="40.894" width="0.127" layer="1"/>
+<wire x1="8.9154" y1="40.894" x2="8.9154" y2="39.37" width="0.127" layer="1"/>
 </signal>
 <signal name="DACA">
@@
 <signal name="CS3">
 <contactref element="J_CS3" pad="1"/>
-<contactref element="UC" pad="20/A6"/>
-<wire x1="7.8486" y1="39.243" x2="7.8486" y2="37.6174" width="0.127" layer="1"/>
-<wire x1="7.8486" y1="37.6174" x2="8.128" y2="37.338" width="0.127" layer="1"/>
-<wire x1="21.59" y1="16.764" x2="22.225" y2="16.764" width="0.127" layer="1"/>
-<wire x1="22.225" y1="16.764" x2="22.225" y2="16.637" width="0.127" layer="1"/>
-<wire x1="22.225" y1="16.637" x2="23.114" y2="15.748" width="0.127" layer="1"/>
-<wire x1="23.114" y1="15.748" x2="23.114" y2="10.795" width="0.127" layer="1"/>
-<wire x1="23.114" y1="10.795" x2="22.606" y2="10.287" width="0.127" layer="1"/>
-<wire x1="22.606" y1="10.287" x2="18.161" y2="10.287" width="0.127" layer="1"/>
-<wire x1="8.128" y1="37.338" x2="8.128" y2="20.32" width="0.127" layer="1"/>
-<wire x1="8.128" y1="20.32" x2="18.161" y2="10.287" width="0.127" layer="1"/>
+<contactref element="UC" pad="21/A7"/>
+<wire x1="18.288" y1="10.668" x2="22.352" y2="10.668" width="0.127" layer="1"/>
+<wire x1="22.352" y1="10.668" x2="22.733" y2="11.049" width="0.127" layer="1"/>
+<wire x1="22.733" y1="11.049" x2="22.733" y2="13.716" width="0.127" layer="1"/>
+<wire x1="22.733" y1="13.716" x2="22.225" y2="14.224" width="0.127" layer="1"/>
+<wire x1="22.225" y1="14.224" x2="21.59" y2="14.224" width="0.127" layer="1"/>
+<wire x1="8.509" y1="38.608" x2="8.509" y2="20.447" width="0.127" layer="1"/>
+<wire x1="8.509" y1="20.447" x2="18.288" y2="10.668" width="0.127" layer="1"/>
+<wire x1="8.509" y1="38.608" x2="7.8486" y2="39.2684" width="0.127" layer="1"/>
+<wire x1="7.8486" y1="39.2684" x2="7.8486" y2="39.37" width="0.127" layer="1"/>
 </signal>
 <signal name="VI_LP">
@@
 <wire x1="17.907" y1="18.161" x2="16.51" y2="16.764" width="0.127" layer="1"/>
 </signal>
-<signal name="CS2">
-<contactref element="J_CS2" pad="1"/>
-<contactref element="UC" pad="21/A7"/>
-<wire x1="7.8486" y1="40.894" x2="7.8486" y2="40.6654" width="0.127" layer="1"/>
-<wire x1="7.8486" y1="40.6654" x2="8.382" y2="40.132" width="0.127" layer="1"/>
-<wire x1="8.382" y1="40.132" x2="8.382" y2="37.592" width="0.127" layer="1"/>
-<wire x1="8.382" y1="37.592" x2="8.509" y2="37.465" width="0.127" layer="1"/>
-<wire x1="18.288" y1="10.668" x2="22.352" y2="10.668" width="0.127" layer="1"/>
-<wire x1="22.352" y1="10.668" x2="22.733" y2="11.049" width="0.127" layer="1"/>
-<wire x1="22.733" y1="11.049" x2="22.733" y2="13.716" width="0.127" layer="1"/>
-<wire x1="22.733" y1="13.716" x2="22.225" y2="14.224" width="0.127" layer="1"/>
-<wire x1="22.225" y1="14.224" x2="21.59" y2="14.224" width="0.127" layer="1"/>
-<wire x1="8.509" y1="37.465" x2="8.509" y2="20.447" width="0.127" layer="1"/>
-<wire x1="8.509" y1="20.447" x2="18.288" y2="10.668" width="0.127" layer="1"/>
-</signal>
 <signal name="NOGND">
 <polygon width="0.254" layer="2" pour="cutout">
@@
 <wire x1="12.954" y1="53.975" x2="18.034" y2="48.895" width="0.127" layer="1"/>
 </signal>
+<signal name="CS2">
+<contactref element="J_CS2" pad="1"/>
+<contactref element="UC" pad="20/A6"/>
+<wire x1="7.8486" y1="37.6174" x2="8.128" y2="37.338" width="0.127" layer="1"/>
+<wire x1="21.59" y1="16.764" x2="22.225" y2="16.764" width="0.127" layer="1"/>
+<wire x1="22.225" y1="16.764" x2="22.225" y2="16.637" width="0.127" layer="1"/>
+<wire x1="22.225" y1="16.637" x2="23.114" y2="15.748" width="0.127" layer="1"/>
+<wire x1="23.114" y1="15.748" x2="23.114" y2="10.795" width="0.127" layer="1"/>
+<wire x1="23.114" y1="10.795" x2="22.606" y2="10.287" width="0.127" layer="1"/>
+<wire x1="22.606" y1="10.287" x2="18.161" y2="10.287" width="0.127" layer="1"/>
+<wire x1="8.128" y1="37.338" x2="8.128" y2="20.32" width="0.127" layer="1"/>
+<wire x1="8.128" y1="20.32" x2="18.161" y2="10.287" width="0.127" layer="1"/>
+<wire x1="7.8486" y1="37.6174" x2="7.8486" y2="38.2016" width="0.127" layer="1"/>
+<wire x1="7.8486" y1="38.2016" x2="7.874" y2="38.354" width="0.127" layer="1"/>
+<via x="7.874" y="38.354" extent="1-16" drill="0.1778"/>
+<via x="8.382" y="40.132" extent="1-16" drill="0.1778"/>
+<wire x1="7.874" y1="38.354" x2="7.874" y2="39.624" width="0.127" layer="16"/>
+<wire x1="7.874" y1="39.624" x2="8.382" y2="40.132" width="0.127" layer="16"/>
+<wire x1="8.382" y1="40.132" x2="7.8486" y2="40.6654" width="0.127" layer="1"/>
+<wire x1="7.8486" y1="40.6654" x2="7.8486" y2="40.894" width="0.127" layer="1"/>
+</signal>
 </signals>
